File: flight_computer_dev_board/flight_computer_dev_board_rfm98pw/flight_computer_dev_board_rfm98pw.kicad_pcb (KiCad board)
At the start: 4 copper layers, 88 x 94.5 mm, 103 parts, among them IC1 RP2040_QFN56, IC2 AZ1117CH-3.3TRG1, J1 Conn_ARM_JTAG_SWD_10, J2 FC to EPS Connector, J3 Life Makes Lemonade, J4 104031-0811, J5 RJ45_LED_Shielded, J6 Conn_Coaxial, J7 Breakout, J8 USB_B_Micro, SW1 KMR2, SW2 KMR2, U1 SN74AHC1G125DBVR, U2 W5500, U3 MAX706RESA, U4 RFM98PW, U5 RFM9xBreakout, U6 W25Q128JV, U7 LSM6DSOTR, U8 LSM303AGRTR, Y1 12MHZ, Y2 25MHz

Commit message: Flight Computer dev board minor update
Routing:
- net GND: track 151.6 -> 164.8 mm, vias 29 -> 61
- net RF1_ANT: track 9.05 -> 10.5 mm
- net VCC_RF1: track 101.5 -> 102.9 mm
- net RF1_IO4: track 55.6 -> 57.0 mm
- net RF1_IO0: track 53.6 -> 55.1 mm
- net 3.3V: vias 5 -> 11
- added copper zone on In2.Cu, net 3.3V
- added copper zone on In1.Cu, net GND
- removed copper zone on In1.Cu, net 3.3V
- removed copper zone on In2.Cu, net GND
