File: antenna_top_cap_board/antenna_top_cap_V1/antenna_top_cap.kicad_pcb (KiCad board)
At the start: 4 copper layers, 100 x 100 mm, 39 parts, among them IC1 PCT2075DP,118, J1 Battery Charge Bypass, J2 Battery Charge Bypass, J3 Burn_Wire, J4 Breakout, J5 Conn_Coaxial, J8 Breakout, Q1 BSS138, U1 VL6180XV0NR/1, U2 LP5907-2.8V, U3 0433BM15A0001

Commit message: Antenna Top Cap for Development Board
Parts:
- removed the G*** at (191.5, 70.7)
- removed the G*** at (194.3, 94.9)
- removed the G*** at (177.5, 152.9)
- removed the G*** at (176.0, 100.4)
- added D2: Blue, LED_SMD:LED_0603_1608Metric, F.Cu at (118.4, 81.8)
- added D3: Blue, LED_SMD:LED_0603_1608Metric, F.Cu at (118.6, 92.0)
- added D4: Blue, LED_SMD:LED_0603_1608Metric, F.Cu at (212.4, 91.4)
- added D5: Blue, LED_SMD:LED_0603_1608Metric, F.Cu at (212.4, 81.0)
- added G*** (x2): LOGO, LOGO, B.Cu at (189.5, 72.3)
- added J10: USB_B_Micro, FC_DEV_BOARD:MOLEX_105164-0001, B.Cu at (115.5, 81.7)
- added J11: USB_B_Micro, FC_DEV_BOARD:MOLEX_105164-0001, B.Cu at (115.5, 91.8)
- added J12: BM04B-SRSS-TB(LF)(SN), Antenna_board:JST_BM04B-SRSS-TB(LF)(SN), F.Cu at (132.0, 91.4)
- added J13: USB_B_Micro, FC_DEV_BOARD:MOLEX_105164-0001, B.Cu at (215.5, 91.1)
- added J14: BM04B-SRSS-TB(LF)(SN), Antenna_board:JST_BM04B-SRSS-TB(LF)(SN), F.Cu at (198.8, 91.4)
- added J15: USB_B_Micro, FC_DEV_BOARD:MOLEX_105164-0001, B.Cu at (215.5, 80.9)
- added J16: BM04B-SRSS-TB(LF)(SN), Antenna_board:JST_BM04B-SRSS-TB(LF)(SN), F.Cu at (198.8, 81.2)
- added J9: BM04B-SRSS-TB(LF)(SN), Antenna_board:JST_BM04B-SRSS-TB(LF)(SN), F.Cu at (132.1, 81.4)
- added R5: 1K, Resistor_SMD:R_0402_1005Metric, F.Cu at (121.5, 79.6)
- added R6: 1K, Resistor_SMD:R_0402_1005Metric, F.Cu at (121.5, 89.4)
- added R7: 1K, Resistor_SMD:R_0402_1005Metric, F.Cu at (208.9, 94.0)
- added R8: 1K, Resistor_SMD:R_0402_1005Metric, F.Cu at (208.8, 83.3)
- moved G*** 18.9 mm to (194.3, 94.4)
- moved G*** 6.60 mm to (184.4, 154.3)
Routing:
- net GND: track 23.7 -> 104.1 mm, vias 7 -> 11
- net Net-(J10-VBUS): track 0.00 -> 11.9 mm, vias 0 -> 1
- net Net-(J11-VBUS): track 0.00 -> 11.4 mm, vias 0 -> 1
- net Net-(J13-VBUS): track 0.00 -> 11.2 mm, vias 0 -> 1
- net 2.8V: track 161.0 -> 150.0 mm, vias 2 -> 3
- net /2d-: track 0.00 -> 10.8 mm, vias 0 -> 1
- net Net-(J15-VBUS): track 0.00 -> 10.8 mm, vias 0 -> 1
- net /3d-: track 0.00 -> 10.8 mm, vias 0 -> 1
- net /1d-: track 0.00 -> 10.5 mm, vias 0 -> 1
- net /2d+: track 0.00 -> 10.5 mm, vias 0 -> 1
- net /3d+: track 0.00 -> 10.5 mm, vias 0 -> 1
- net /0d-: track 0.00 -> 10.5 mm, vias 0 -> 1
- net /1d+: track 0.00 -> 10.2 mm, vias 0 -> 1
- net /0d+: track 0.00 -> 10.2 mm, vias 0 -> 1
- net Net-(D4-A): track 0.00 -> 3.76 mm
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Other:
- outline, holes or cut-outs redrawn
- board text added: "BEFORE FLIGHT: 1.) Ensure WDT Resistor is Populated 2.) Check Burnwire Setting 3.) Remove Inhibit Boots 4a.) Don't Panic 4b.) Integrate Satellite Quickly! 5.) Remove RBF Pin 6.) Celebrate! 7.) FiFi"
- board text added: "Camera USB"
- board text added: "EPS USB"
- board text added: "FC USB"
- board text added: "Payload USB"
- board text added: "The Spacecraft Company LLC"
- board text removed: "As seen on-orbit:"
- board text removed: "BEFORE FLIGHT: 1.) Ensure R2 is Populated 2.) Check Burnwire Setting 3.) Remove Inhibit Boots 4a.) Don't Panic 4b.) Integrate Satellite Quickly! 5.) Remove RBF Pin 6.) Celebrate! 7.) FiFi"
- board text removed: "BRONCO SPACE Educational Product For Instructional Use Only"
- board text removed: "This CubeSat was designed entirely by STUDENTS at California State Polytechnic University, Pomona"
