File: antenna_top_cap_board/antenna_top_cap_V1/antenna_top_cap.kicad_pcb (KiCad board)
At the start: 4 copper layers, 100 x 100 mm, 61 parts, among them IC1 PCT2075DP,118, J1 Battery Charge Bypass, J10 USB_B_Micro, J11 USB_B_Micro, J12 BM04B-SRSS-TB(LF)(SN), J13 USB_B_Micro, J14 BM04B-SRSS-TB(LF)(SN), J15 USB_B_Micro, J16 BM04B-SRSS-TB(LF)(SN), J17 BM04B-SRSS-TB(LF)(SN), J18 BM04B-SRSS-TB(LF)(SN), J2 Battery Charge Bypass, J3 Burn_Wire, J4 BM04B-SRSS-TB(LF)(SN), J5 Conn_Coaxial, J8 BM04B-SRSS-TB(LF)(SN), J9 BM04B-SRSS-TB(LF)(SN), Q1 BSS138, U1 VL6180XV0NR/1, U2 LP5907-2.8V, U3 0433BM15A0001, U4 AS193-73LF, U5 RFM98PW, U6 RFM9xBreakout

Commit message: Fixed Antenna Board
Parts:
- moved J5 5.53 mm to (164.5, 117.7)
- moved J3 4.34 mm to (144.7, 112.8), turned to 180 degrees
- moved R1 2.18 mm to (160.4, 102.7), turned to 45 degrees
Routing:
- net SCL1: track 32.3 -> 41.6 mm, vias 2 -> 4
- net Net-(J3-Pin_1): track 23.2 -> 15.2 mm
- net GND: track 178.2 -> 171.1 mm, vias 40 -> 31
- net Balun: track 33.3 -> 27.0 mm
- net Net-(J3-Pin_2): track 23.4 -> 20.4 mm
- net 3.3V: track 42.9 -> 45.6 mm
- net Net-(D1-A): track 0.00 -> 1.75 mm
