File: flight_computer_dev_board/flight_computer_dev_board_sx1276/flight_computer_dev_board_sx1276.kicad_pcb (KiCad board)
At the start: 4 copper layers, 88 x 94.5 mm, 185 parts, among them IC1 RP2040_QFN56, IC2 AZ1117CH-3.3TRG1, J1 Conn_ARM_JTAG_SWD_10, J2 USB_B_Micro, J3 RJ45_LED_Shielded, J4 Breakout, J5 Life Makes Lemonade, J6 FC to EPS Connector, J7 104031-0811, J8 Conn_Coaxial, J9 Conn_Coaxial, SW1 KMR2, SW2 KMR2, U1 LSM6DSOTR, U10 4259-63, U11 TRF37A73IDSGR, U12 TRF37A73IDSGR, U13 TRF37A73IDSGR, U14 TRF37A73IDSGR, U2 MAX706RESA, U3 LSM303AGRTR, U4 SN74AHC1G125DBVR, U5 W25Q128JV, U6 W5500, U7 SX1276IMLTRT, U8 74LVC1G04W5-7, U9 4259-63, Y1 12MHZ, Y2 Crystal_GND24, Y3 25MHz

Commit message: sx1276 update
Parts:
- removed U12, U14: TRF37A73IDSGR, Package_DFN_QFN:DFN-8-1EP_2x2mm_P0.5mm_EP0.6x1.2mm
- C79, C83, C89, C93: value 1nf -> 100nf
- C80, C90: value 1nf -> 1uf
- C82, C92: value 1nf -> 68pf
- L14, L16: value 100nH -> 470nH
Connections:
- C80 pad 2: +3.3VA -> VCC_RF1
- C81 pad 1: +3.3VA -> VCC_RF1
- C82 pad 1: +3.3VA -> VCC_RF1
- C90 pad 2: +3.3VA -> VCC_RF1
- C91 pad 1: +3.3VA -> VCC_RF1
- C92 pad 1: +3.3VA -> VCC_RF1
- J3 pad 11: YELLOWLED -> GREENLED
- J3 pad 9: GREENLED -> YELLOWLED
- J6 pad 6: GND -> +3V3
- L14 pad 2: +3.3VA -> VCC_RF1
- L16 pad 2: +3.3VA -> VCC_RF1
Routing:
- net +3V3: track 48.0 -> 49.2 mm, vias 11 -> 12
- net GND: track 119.5 -> 118.3 mm, vias 33 -> 32
