File: flight_computer_dev_board/flight_computer_dev_board_sx1276/flight_computer_dev_board_sx1276.kicad_sch (KiCad schematic)
At the start: 181 parts, among them IC1 RP2040_QFN56, IC2 AZ1117CH-3.3TRG1, J1 Conn_ARM_JTAG_SWD_10, J2 USB_B_Micro, J3 RJ45_LED_Shielded, J4 Breakout, J5 Life Makes Lemonade, J6 FC to EPS Connector, J7 104031-0811, J8 Conn_Coaxial, J9 Conn_Coaxial, SW1 KMR2, SW2 KMR2, U1 LSM6DSOTR, U10 4259-63, U11 TRF37A73IDSGR, U12 TRF37A73IDSGR, U13 TRF37A73IDSGR, U14 TRF37A73IDSGR, U2 MAX706RESA, U3 LSM303AGRTR, U4 SN74AHC1G125DBVR, U5 W25Q128JV, U6 W5500, U7 SX1276IMLTRT, U8 74LVC1G04W5-7, U9 4259-63, Y1 12MHZ, Y1 25MHz, Y2 Crystal_GND24

Commit message: sx1276 update
Parts:
- removed C14 (x4): 1nf, Capacitor_SMD:C_0402_1005Metric, symbol Adafruit Ethernet FeatherWing-eagle-import:CAP_CERAMIC0805-NOOUTLINE
- removed U12, U14: TRF37A73IDSGR, Package_DFN_QFN:DFN-8-1EP_2x2mm_P0.5mm_EP0.6x1.2mm, symbol TRF37A73IDSGR:TRF37A73IDSGR
- added C14: 1nf, Capacitor_SMD:C_0402_1005Metric, symbol Adafruit Ethernet FeatherWing-eagle-import:CAP_CERAMIC0805-NOOUTLINE
- added C14: 68pf, Capacitor_SMD:C_0402_1005Metric, symbol Adafruit Ethernet FeatherWing-eagle-import:CAP_CERAMIC0805-NOOUTLINE
- added C14: 100nf, Capacitor_SMD:C_0402_1005Metric, symbol Adafruit Ethernet FeatherWing-eagle-import:CAP_CERAMIC0805-NOOUTLINE
- added C14: 1uf, Capacitor_SMD:C_0402_1005Metric, symbol Adafruit Ethernet FeatherWing-eagle-import:CAP_CERAMIC0805-NOOUTLINE
- added U12, U15: ADL5536ARKZ-R7, Package_TO_SOT_SMD:SOT-89-3, symbol ADL5536:ADL5536ARKZ-R7
- C14: value 1nf -> 1uf
- C14: value 1nf -> 100nf
- C14: value 1nf -> 68pf
- L14, L16: value 100nH -> 470nH
Connections:
- net +3.3VA: no longer C14.1, C14.1, C14.2, L14.2, L16.2
- net +3V3: now also J6.6 (Pin_6)
- net GND: now also C14.1, C14.2, C14.2, U12.2 (GND), U15.2 (GND); no longer J6.6 (Pin_6)
- net GREENLED: now also J3.11; no longer J3.9
- net HIGH_OUT2: now also C14.2
- net RF_CONTROL: now also U7.20 (RXTX/RFMOD); no longer IC1.40 (GPIO28/AD2)
- net VCC_RF1: now also C14.1, C14.1, C14.2, L14.2, L16.2, C14.1, C14.1, C14.2
- net YELLOWLED: now also J3.9; no longer J3.11
- net at L16.1: now also C14.1, U12.3 (REFOUT)
- net at C14.2: now also U15.1 (REFIN)
- net at C14.1, L14.1: now also U15.3 (REFOUT)
- net at C14.2: now also U12.1 (REFIN)
Other:
- moved on the sheet: C14, L14
