File: flight_computer_dev_board/flight_computer_dev_board_rfm98pw/V1/flight_computer_dev_board_rfm98pw.kicad_pcb (KiCad board)
At the start: 4 copper layers, 88 x 94.5 mm, 103 parts, among them IC1 RP2040_QFN56, IC2 AZ1117CH-3.3TRG1, J1 Conn_ARM_JTAG_SWD_10, J2 FC to EPS Connector, J3 Life Makes Lemonade, J4 104031-0811, J5 RJ45_LED_Shielded, J6 Conn_Coaxial, J7 Breakout, J8 USB_B_Micro, SW1 KMR2, SW2 KMR2, U1 SN74AHC1G125DBVR, U2 W5500, U3 MAX706RESA, U4 RFM98PW, U5 RFM9xBreakout, U6 W25Q128JV, U7 LSM6DSOTR, U8 LSM303AGRTR, Y1 12MHZ, Y2 25MHz

Commit message: sx1276 update
Parts:
- added J9: BM04B-SRSS-TB(LF)(SN), FC_DEV_BOARD:JST_BM04B-SRSS-TB(LF)(SN), F.Cu at (222.5, 74.4)
- moved U6 0.58 mm to (215.8, 74.7)
Connections:
- J2 pad 6: GND -> 3.3V
- J5 pad 11: YELLOWLED -> GREENLED
- J5 pad 9: GREENLED -> YELLOWLED
Routing:
- net USB_D+: track 5.79 -> 19.3 mm, vias 2 -> 3
- net USB_D-: track 5.77 -> 18.5 mm, vias 2 -> 3
- net GND: track 164.8 -> 173.3 mm
- net VBUS: track 70.9 -> 77.9 mm, vias 4 -> 5
- net GREENLED: track 52.1 -> 46.4 mm
- net YELLOWLED: track 46.8 -> 50.9 mm
- net 3.3V: track 48.0 -> 51.9 mm, vias 11 -> 13
- net /QSPI_DATA[1]: track 14.1 -> 13.4 mm
- net /QSPI_CS: track 23.9 -> 24.4 mm

Commit message: rfm98pw dev board V1 update
Parts:
- removed D6: NSR0320, Diode_SMD:D_SOD-323F
- added C37: 22pf, Capacitor_SMD:C_0402_1005Metric, F.Cu at (172.7, 120.2)
- added C38: 22pf, Capacitor_SMD:C_0402_1005Metric, F.Cu at (171.6, 115.7)
- added C39: 47pf, Capacitor_SMD:C_0402_1005Metric, F.Cu at (162.9, 129.4)
- added C40: 47pf, Capacitor_SMD:C_0402_1005Metric, F.Cu at (168.5, 129.4)
- added C41: 10uf, Capacitor_SMD:C_0603_1608Metric, F.Cu at (180.2, 124.8)
- added C42: 1uf, Capacitor_SMD:C_0603_1608Metric, F.Cu at (178.6, 124.0)
- added C43: 10uf, Capacitor_SMD:C_0603_1608Metric, F.Cu at (175.8, 120.8)
- added D8: PESD1CAN, Package_TO_SOT_SMD:SOT-23-3, F.Cu at (165.7, 127.9)
- added G***: LOGO, LOGO, B.Cu at (183.9, 66.5)
- added G***: LOGO, LOGO, B.Cu at (191.0, 128.6)
- added J10: BM04B-SRSS-TB(LF)(SN), FC_DEV_BOARD:JST_BM04B-SRSS-TB(LF)(SN), F.Cu at (185.5, 80.0)
- added J11: BM04B-SRSS-TB(LF)(SN), FC_DEV_BOARD:JST_BM04B-SRSS-TB(LF)(SN), F.Cu at (181.9, 90.2)
- added J12: BM04B-SRSS-TB(LF)(SN), FC_DEV_BOARD:JST_BM04B-SRSS-TB(LF)(SN), B.Cu at (181.9, 95.3)
- added J13: Breakout, Connector_JST:JST_SH_SM04B-SRSS-TB_1x04-1MP_P1.00mm_Horizontal, F.Cu at (164.6, 133.4)
- added JP7: SolderJumper_3_Open, Jumper:SolderJumper-3_P1.3mm_Open_RoundedPad1.0x1.5mm_NumberLabels, F.Cu at (171.6, 80.0)
- added JP8: SolderJumper_2_Open, Jumper:SolderJumper-2_P1.3mm_Open_RoundedPad1.0x1.5mm, F.Cu at (199.9, 115.0)
- added R23: 10k, Resistor_SMD:R_0603_1608Metric, F.Cu at (161.0, 114.2)
- added R24: 10k, Resistor_SMD:R_0603_1608Metric, F.Cu at (158.3, 119.0)
- added R25: 10k, Resistor_SMD:R_0603_1608Metric, F.Cu at (169.3, 123.0)
- added R26: 120, Resistor_SMD:R_0603_1608Metric, F.Cu at (165.7, 125.1)
- added R27: 10k, Resistor_SMD:R_0603_1608Metric, F.Cu at (174.9, 126.6)
- added R28: 10k, Resistor_SMD:R_0603_1608Metric, F.Cu at (184.4, 106.6)
- added TP3: RESET, TestPoint:TestPoint_Loop_D1.80mm_Drill1.0mm_Beaded, F.Cu at (154.9, 118.3)
- added TP4: Standby, TestPoint:TestPoint_Loop_D1.80mm_Drill1.0mm_Beaded, F.Cu at (170.9, 126.8)
- added U10: AP3602AKTR-G1, Package_TO_SOT_SMD:SOT-23-6, F.Cu at (175.5, 124.0)
- added U9: MCP25625-E/ML, Package_DFN_QFN:QFN-28-1EP_6x6mm_P0.65mm_EP4.25x4.25mm, F.Cu at (164.7, 119.6)
- added Y3: 16MHZ 12 pf, Crystal:Crystal_SMD_2520-4Pin_2.5x2.0mm, F.Cu at (171.6, 118.0)
- J5: moved to F.Cu
- moved C19 12.9 mm to (172.4, 96.3)
- moved C18 10.8 mm to (172.4, 95.3)
- moved R19 10.3 mm to (174.1, 95.3), turned to 90 degrees
- moved R18 8.82 mm to (175.6, 94.4), turned to 90 degrees
- moved C36 6.14 mm to (172.4, 92.8), turned to 0 degrees
- moved R14 5.39 mm to (173.0, 87.4)
- moved J5 4.86 mm to (168.7, 87.4), turned to -90 degrees
- moved R13 4.44 mm to (180.5, 78.5), turned to 90 degrees
- moved C17 3.40 mm to (172.4, 91.8)
- moved R16 2.33 mm to (173.0, 89.0)
- moved R17 0.94 mm to (173.0, 90.5)
Connections:
- net SPI0_CS1 renamed SPI1_CS1
- C14 pad 2: VCC_RF1 -> RF_VCC
- C27 pad 1: 3.3V -> 3v3_prime
- C28 pad 1: 3.3V -> 3v3_prime
- FB1 pad 1: 3.3V -> 3v3_prime
- IC1 pad 11: SPI1_MISO -> SPI0_MISO
- IC1 pad 12: SPI1_CS0 -> SPI0_CS0
- IC1 pad 13: SPI1_SCK -> SPI0_SCK
- IC1 pad 14: SPI1_MOSI -> SPI0_MOSI
- IC1 pad 27: SPI0_MISO -> SPI1_MISO
- IC1 pad 28: SPI0_CS0 -> SPI1_CS0
- IC1 pad 29: SPI0_SCK -> SPI1_SCK
- IC1 pad 30: SPI0_MOSI -> SPI1_MOSI
- IC1 pad 40: /A2 -> SPI1_CS2
- J4 pad 2: SPI0_CS0 -> SPI1_CS0
- J4 pad 3: SPI0_MOSI -> SPI1_MOSI
- J4 pad 5: SPI0_SCK -> SPI1_SCK
- J4 pad 7: SPI0_MISO -> SPI1_MISO
- JP1 pad 2: Net-(D6-K) -> 3v3 Spec
- R13 pad 2: SPI1_CS0 -> SPI0_CS0
- R15 pad 1: SPI0_CS0 -> SPI1_CS0
- R22 pad 5: 3.3V -> 3v3_prime
- R22 pad 6: 3.3V -> 3v3_prime
- R22 pad 7: 3.3V -> 3v3_prime
- R22 pad 8: 3.3V -> 3v3_prime
- U1 pad 4: SPI0_MISO -> SPI1_MISO
- U2 pad 28: 3.3V -> 3v3_prime
- U2 pad 33: SPI0_SCK -> SPI1_SCK
- U2 pad 35: SPI0_MOSI -> SPI1_MOSI
- U2 pad 37: unconnected-(U2-RSTN-Pad37) -> Net-(U2-RSTN)
- U4 pad 10: SPI1_MISO -> SPI0_MISO
- U4 pad 11: SPI1_MOSI -> SPI0_MOSI
- U4 pad 12: SPI1_SCK -> SPI0_SCK
- U4 pad 13: SPI1_CS0 -> SPI0_CS0
- U4 pad 5: VCC_RF1 -> RF_VCC
- U5 pad 13: VCC_RF1 -> RF_VCC
- U5 pad 2: SPI1_MISO -> SPI0_MISO
- U5 pad 3: SPI1_MOSI -> SPI0_MOSI
- U5 pad 4: SPI1_SCK -> SPI0_SCK
- U5 pad 5: SPI1_CS0 -> SPI0_CS0
Routing:
- net SPI1_CS2: track 0.00 -> 72.4 mm, vias 0 -> 5
- net SPI1_MISO: track 35.3 -> 96.0 mm, vias 2 -> 9
- net SPI1_MOSI: track 37.1 -> 91.9 mm, vias 2 -> 8
- net SPI1_SCK: track 38.9 -> 89.6 mm, vias 2 -> 8
- net GND: track 173.3 -> 215.1 mm, vias 61 -> 74
- net 3v3_prime: track 0.00 -> 38.1 mm, vias 0 -> 2
- net RF_VCC: track 0.00 -> 19.2 mm
- net SPI0_MOSI: track 61.6 -> 44.9 mm
- net SPI0_MISO: track 61.7 -> 45.3 mm, vias 5 -> 2
- net SPI0_CS0: track 46.4 -> 61.5 mm, vias 5 -> 4
- net RX-: track 41.7 -> 27.3 mm
- net SPI0_SCK: track 59.7 -> 48.4 mm
- net TXCAN: track 0.00 -> 11.0 mm, vias 0 -> 2
- net CANH: track 0.00 -> 10.7 mm
- net CANL: track 0.00 -> 10.7 mm
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Other:
- board text added: "5V"
- board text added: "Always has been!"
- board text added: "CAN BUS"
- board text added: "EPS DIRECT CONTROL"
- board text added: "I2C STEMMA QWIIK"
- board text added: "M1 The Crab Nebula"
- board text added: "RF Power Jumper"
- board text added: "SPI"
- board text added: "Standby"
- board text added: "USB"
- board text added: "USB Breakout"
- board text added: "Wait its all open source?"
