File: flight_computer_dev_board/flight_computer_dev_board_rfm98pw/V1/flight_computer_dev_board_rfm98pw.kicad_sch (KiCad schematic)
At the start: 99 parts, among them IC1 RP2040_QFN56, IC2 AZ1117CH-3.3TRG1, J1 Conn_ARM_JTAG_SWD_10, J2 FC to EPS Connector, J3 Life Makes Lemonade, J4 104031-0811, J5 RJ45_LED_Shielded, J6 Conn_Coaxial, J7 Breakout, J8 USB_B_Micro, SW1 KMR2, SW2 KMR2, U1 SN74AHC1G125DBVR, U2 W5500, U3 MAX706RESA, U4 RFM98PW, U5 RFM9xBreakout, U6 W25Q128JV, U7 LSM6DSOTR, U8 LSM303AGRTR, Y1 12MHZ, Y1 25MHz

Commit message: sx1276 update
Parts:
- added J9: BM04B-SRSS-TB(LF)(SN), FC_DEV_BOARD:JST_BM04B-SRSS-TB(LF)(SN), symbol BM04B-SRSS-TB_LF__SN_:BM04B-SRSS-TB(LF)(SN)
Connections:
- net +3V3: now also J2.6 (Pin_6)
- net GND: now also J9.4, J9.S1 (SHIELD), J9.S2 (SHIELD); no longer J2.6 (Pin_6)
- net GREENLED: now also J5.11; no longer J5.9
- net USB_D+: now also J9.3
- net USB_D-: now also J9.2
- net VBUS: now also J9.1
- net YELLOWLED: now also J5.9; no longer J5.11

Commit message: rfm98pw dev board V1 update
Parts:
- removed D6: NSR0320, Diode_SMD:D_SOD-323F, symbol Diode:1SS355VM
- added C13 (x2): 22pf, Capacitor_SMD:C_0402_1005Metric, symbol Adafruit Ethernet FeatherWing-eagle-import:CAP_CERAMIC0603_NO
- added C13 (x2): 47pf, Capacitor_SMD:C_0402_1005Metric, symbol Adafruit Ethernet FeatherWing-eagle-import:CAP_CERAMIC0603_NO
- added C13: 1uf, Capacitor_SMD:C_0603_1608Metric, symbol Adafruit Ethernet FeatherWing-eagle-import:CAP_CERAMIC0603_NO
- added C13 (x2): 10uf, Capacitor_SMD:C_0603_1608Metric, symbol Adafruit Ethernet FeatherWing-eagle-import:CAP_CERAMIC0603_NO
- added D8: PESD1CAN, Package_TO_SOT_SMD:SOT-23-3, symbol PESD1CAN:PESD1CAN
- added J10, J11, J12: BM04B-SRSS-TB(LF)(SN), FC_DEV_BOARD:JST_BM04B-SRSS-TB(LF)(SN), symbol BM04B-SRSS-TB_LF__SN_:BM04B-SRSS-TB(LF)(SN)
- added J13: Breakout, Connector_JST:JST_SH_SM04B-SRSS-TB_1x04-1MP_P1.00mm_Horizontal, symbol Connector_Generic:Conn_01x04
- added JP7: SolderJumper_3_Open, Jumper:SolderJumper-3_P1.3mm_Open_RoundedPad1.0x1.5mm_NumberLabels, symbol Jumper:SolderJumper_3_Open
- added JP8: SolderJumper_2_Open, Jumper:SolderJumper-2_P1.3mm_Open_RoundedPad1.0x1.5mm, symbol Jumper:SolderJumper_2_Open
- added R23, R24, R25, R27, R28: 10k, Resistor_SMD:R_0603_1608Metric, symbol mainboard:10KOHM-1_10W-1%(0603)0603
- added R26: 120, Resistor_SMD:R_0603_1608Metric, symbol mainboard:10KOHM-1_10W-1%(0603)0603
- added TP3: RESET, TestPoint:TestPoint_Loop_D1.80mm_Drill1.0mm_Beaded, symbol Connector:TestPoint
- added TP4: Standby, TestPoint:TestPoint_Loop_D1.80mm_Drill1.0mm_Beaded, symbol Connector:TestPoint
- added U10: AP3602AKTR-G1, Package_TO_SOT_SMD:SOT-23-6, symbol AP3602:AP3602AKTR-G1
- added U9: MCP25625-E/ML, Package_DFN_QFN:QFN-28-1EP_6x6mm_P0.65mm_EP4.25x4.25mm, symbol MCP25625-E_ML:MCP25625-E/ML
- added Y3: 16MHZ 12 pf, Crystal:Crystal_SMD_2520-4Pin_2.5x2.0mm, symbol Adafruit ItsyBitsy RP2040-eagle-import:CRYSTAL2.5X2.0
Connections:
- net +3V3: now also C13.2, J11.1, J12.1, J13.2 (Pin_2), JP7.3 (B), JP8.1 (A), R23.1, R24.1, R27.1, U10.5 (VIN), U9.11 (VIO), U9.3 (VDD@1); no longer C14.1, C15.1, FB1.1, R22.5 (R4.2), R22.6 (R3.2), R22.7 (R2.2), R22.8 (R1.2), U2.28 (VDD)
- net 3v3 Spec: now also JP1.2 (B)
- net GND: now also C13.1, C13.1, C13.1, C13.2, C13.2, C13.2, D8.3, J10.S1 (SHIELD), J10.S2 (SHIELD), J11.2, J11.4, J11.S1 (SHIELD), J11.S2 (SHIELD), J12.2, J12.4, J12.S1 (SHIELD), J12.S2 (SHIELD), J13.1 (Pin_1), R25.1, U10.2 (GND), U9.18 (VSS@1), U9.22 (GND), U9.29 (GND@1)
- net SPI0_CS0: now also IC1.12 (GPIO9), R13.2, U4.13 (NSS), U5.5 (CS), J10.1; no longer IC1.28 (GPIO17), J4.2 (CD/DAT3), R15.1
- net SPI0_MISO: now also IC1.11 (GPIO8), U4.10 (MISO), U5.2 (MISO), J10.4; no longer IC1.27 (GPIO16), J4.7 (DAT0), U1.4 (Y)
- net SPI0_MOSI: now also IC1.14 (GPIO11), U4.11 (MOSI), U5.3 (MOSI), J10.3; no longer IC1.30 (GPIO19), J4.3 (CMD), U2.35 (MOSI)
- net SPI0_SCK: now also IC1.13 (GPIO10), U4.12 (SCK), U5.4 (SCK), J10.2; no longer IC1.29 (GPIO18), J4.5 (CLK), U2.33 (SCLK)
- net SPI1_CS0: now also IC1.28 (GPIO17), J4.2 (CD/DAT3), R15.1; no longer IC1.12 (GPIO9), R13.2, U4.13 (NSS), U5.5 (CS)
- net SPI1_MISO: now also IC1.27 (GPIO16), J4.7 (DAT0), U1.4 (Y), U9.28 (SO); no longer IC1.11 (GPIO8), U4.10 (MISO), U5.2 (MISO)
- net SPI1_MOSI: now also IC1.30 (GPIO19), J4.3 (CMD), U2.35 (MOSI), U9.27 (SI); no longer IC1.14 (GPIO11), U4.11 (MOSI), U5.3 (MOSI)
- net SPI1_SCK: now also IC1.29 (GPIO18), J4.5 (CLK), U2.33 (SCLK), U9.26 (SCK); no longer IC1.13 (GPIO10), U4.12 (SCK), U5.4 (SCK)
- net VCC_RF1: now also J11.3, J12.3, JP7.1 (A); no longer C14.2, U4.5 (VCC), U5.13 (3V3)
- net at U2.37 (RSTN): now also R28.2
- net A2 renamed SPI1_CS2
- net SPI1_CS2: now also R23.2, U9.1 (CS)
- net SPI0_CS1 renamed SPI1_CS1
- new net: C13.1, U9.20 (OSC2), Y3.1
- new net: R25.2, TP4.1, U9.15 (STBY)
- new net: C13.1, U10.4 (C-)
- new net: C13.2, U10.6 (C+)
- new net: R24.2, TP3.1, U9.2 (RESET)
- new net: C13.1, U9.21 (OSC1), Y3.3 (2)
- new net: R27.2, U10.3 (*SHDN)
- new net +5V: C13.2, U10.1 (VOUT), U9.19 (VDDA)
- new net 3v3_prime: C14.1, C15.1, FB1.1, JP8.2 (B), R22.5 (R4.2), R22.6 (R3.2), R22.7 (R2.2), R22.8 (R1.2), R28.1, U2.28 (VDD)
- new net CANH: C13.2, D8.2, J13.4 (Pin_4), R26.2, U9.13 (CANH)
- new net CANL: C13.1, D8.1, J13.3 (Pin_3), R26.1, U9.12 (CANL)
- new net RF_VCC: C14.2, JP7.2 (C), U4.5 (VCC), U5.13 (3V3)
- new net RXCAN: U9.10 (RXD), U9.5 (RXCAN)
- new net TXCAN: U9.16 (TXD), U9.4 (TXCAN)
- no-connect marks 33 -> 41
