File: Camera_board_v1/camera_v1.kicad_pcb (KiCad board)
At the start: 2 copper layers, 21.4 x 36.6 mm, 27 parts, among them J1 Conn_01x01, J10 I2C1 Breakout, J7 FC Connector, J8 I2C1 Breakout, J9 I2C1 Breakout, U2 TLV74315, U3 TLV74328, X1 CAMERA_OV2640

Commit message: Big Update of In Dev Boards
Mid Term update for all the boards being developed for use by the Irvington Team on Pleiades - Orpheus
Parts:
- removed J10: I2C1 Breakout, Connector_PinHeader_2.54mm:PinHeader_1x04_P2.54mm_Vertical
- removed J9: I2C1 Breakout, Connector_JST:JST_SH_BM04B-SRSS-TB_1x04-1MP_P1.00mm_Vertical
- added G***: LOGO, LOGO, B.Cu at (157.5, 126.4)
- added J2: Conn_01x05, Connector_PinHeader_2.54mm:PinHeader_1x05_P2.54mm_Vertical, F.Cu at (153.7, 105.7)
- added Q1: BSS83P, Package_TO_SOT_SMD:SOT-23, F.Cu at (151.5, 110.9)
- added Q2: BSS138, Package_TO_SOT_SMD:SOT-23, F.Cu at (151.5, 114.5)
- added R1: 10K, Resistor_SMD:R_0603_1608Metric, F.Cu at (154.3, 112.6)
Routing:
- net pwr_in: track 0.00 -> 14.4 mm, vias 0 -> 1
- net pwr_ctrl: track 0.00 -> 10.6 mm, vias 0 -> 1
- net Net-(Q1-G): track 0.00 -> 7.98 mm
- net +3V3: track 31.0 -> 28.0 mm, vias 6 -> 4
- net SDA1: track 42.2 -> 40.8 mm
- net SCL1: track 45.2 -> 44.3 mm
- net GND: track 36.4 -> 37.0 mm
- added copper zone on B.Cu, net pwr_ctrl
- added copper zone on F.Cu, net pwr_ctrl
- added copper zone on B.Cu, net pwr_in
- added copper zone on F.Cu, net pwr_in
- removed copper zone on B.Cu, net +3V3
Other:
- board text added: "I2C Breakout"
- board text added: "Symmetry, hardly know her"
- board text added: "ctrl"
- board text added: "pwr in"
- board text removed: "3V3"
- board text removed: "I2C Breakouts"

Commit message: Before Mirror
Routing:
- net SCL1: track 44.3 -> 39.4 mm
- net SDA1: track 40.8 -> 37.2 mm
- net Net-(J1-Pin_1): track 3.07 -> 0.00 mm
- net 2.8V: track 17.2 -> 15.6 mm
- net AGND: track 1.85 -> 0.45 mm
Changed lines of the file:
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@@
   (segment (start 152.7912 132.3788) (end 152.7912 130.611635) (width 0.1524) (layer "F.Cu") (net 3))
   (segment (start 152.79 122.4375) (end 152.8 122.4275) (width 0.1524) (layer "F.Cu") (net 3))
-  (segment (start 151.83 133.34) (end 151.83 134.9) (width 0.1524) (layer "F.Cu") (net 3))
   (via (at 152.721871 130.542306) (size 0.56) (drill 0.3) (layers "F.Cu" "B.Cu") (net 3))
   (via (at 152.79 123.3) (size 0.56) (drill 0.3) (layers "F.Cu" "B.Cu") (net 3))
@@
   (segment (start 162.153717 131.1938) (end 166.1738 131.1938) (width 0.1524) (layer "B.Cu") (net 4))
   (segment (start 150.51 133.18) (end 150.83 133.5) (width 0.1524) (layer "F.Cu") (net 5))
-  (segment (start 150.83 133.5) (end 150.83 134.9) (width 0.1524) (layer "F.Cu") (net 5))
-  (segment (start 148.45 132.61) (end 150.33 134.49) (width 0.1524) (layer "F.Cu") (net 6))
-  (segment (start 150.33 134.49) (end 150.33 134.9) (width 0.1524) (layer "F.Cu") (net 6))
   (segment (start 161.727738 131.05) (end 162.2862 130.491538) (width 0.1524) (layer "F.Cu") (net 7))
   (segment (start 161.26 131.05) (end 161.727738 131.05) (width 0.1524) (layer "F.Cu") (net 7))
@@
   (segment (start 154.8676 133.26) (end 153.83 134.2976) (width 0.1524) (layer "F.Cu") (net 21))
   (segment (start 155.11 133.26) (end 154.8676 133.26) (width 0.1524) (layer "F.Cu") (net 21))
-  (segment (start 148.76 134.43) (end 149.9062 135.5762) (width 0.1524) (layer "F.Cu") (net 24))
   (segment (start 158.080841 112.8575) (end 159.05 112.8575) (width 0.1524) (layer "F.Cu") (net 24))
-  (segment (start 151.2562 135.5762) (end 151.33 135.5024) (width 0.1524) (layer "F.Cu") (net 24))
   (segment (start 150.5043 117.14) (end 153.798341 117.14) (width 0.1524) (layer "F.Cu") (net 24))
-  (segment (start 151.33 135.5024) (end 151.33 134.9) (width 0.1524) (layer "F.Cu") (net 24))
   (segment (start 159.05 112.8575) (end 159.427738 112.8575) (width 0.1524) (layer "F.Cu") (net 24))
   (segment (start 160.12 108.48) (end 159.69294 108.05294) (width 0.1524) (layer "F.Cu") (net 24))
-  (segment (start 149.9062 135.5762) (end 151.2562 135.5762) (width 0.1524) (layer "F.Cu") (net 24))
   (segment (start 160.12 112.165238) (end 160.12 108.48) (width 0.1524) (layer "F.Cu") (net 24))
   (segment (start 153.798341 117.14) (end 158.080841 112.8575) (width 0.1524) (layer "F.Cu") (net 24))
@@
   (segment (start 158.582473 111.8575) (end 159.05 111.8575) (width 0.1524) (layer "F.Cu") (net 25))
   (segment (start 161.11326 107.49674) (end 161.31 107.3) (width 0.1524) (layer "F.Cu") (net 25))
-  (segment (start 151.9038 135.9286) (end 152.33 135.5024) (width 0.1524) (layer "F.Cu") (net 25))
-  (segment (start 148.6886 135.9286) (end 151.9038 135.9286) (width 0.1524) (layer "F.Cu") (net 25))
   (segment (start 154.159973 116.28) (end 158.582473 111.8575) (width 0.1524) (layer "F.Cu") (net 25))
   (segment (start 161.31 107.3) (end 161.31 105.8532) (width 0.1524) (layer "F.Cu") (net 25))
-  (segment (start 148.355 135.595) (end 148.6886 135.9286) (width 0.1524) (layer "F.Cu") (net 25))
-  (segment (start 152.33 135.5024) (end 152.33 134.9) (width 0.1524) (layer "F.Cu") (net 25))
   (segment (start 159.05 111.8575) (end 159.05 107.909294) (width 0.1524) (layer "F.Cu") (net 25))
   (segment (start 159.05 107.909294) (end 159.462554 107.49674) (width 0.1524) (layer "F.Cu") (net 25))
