File: battery_board_v3/Battery_Board_V3a_with_lt3652/Battery_Board_V3a.kicad_sch (KiCad schematic)
At the start: 201 parts, among them IC2 PCT2075DP,118, IC3 RP2040_QFN56, IC4 LT3652IMSE#PBF, J1 Bypass, J10 Jetson, J11 BM04B-SRSS-TB(LF)(SN), J14 Solar, J15 FC, J16 I2C Multiplexer Breakout, J17 ISS Foot, J18 Screw_Terminal_01x02, J19 BM04B-SRSS-TB(LF)(SN), J2 Heater, J20 CAN1, J21 BM04B-SRSS-TB(LF)(SN), J22 CAN2, J23 Conn_ARM_JTAG_SWD_10, J24 USB_B_Micro, J25 Life Makes Lemonade, J26 BM04B-SRSS-TB(LF)(SN), J27 I2C0 Breakout, J3 BURN, J4 CHARGE, J5 Foot0, J6 Foot1, J7 Foot2, J8 Foot3, J9 RBF, K1 APAN3105, Q1 IRF7458, Q10 IRLML2803, Q11 NDS8434, Q2 IRF7458, Q3 MBT2222ADW1T1, Q4 MMBT2222AT, Q5 MBT2222ADW1T1, Q6 IRLML2803, Q7 IRLML2803, Q8 NDS8434, Q9 NDS8434, SW1 KMR2, SW2 KMR2, U1 R5460N208AA, U10 TLVH431 DBZ SOT-23, U11 MCP25625-E/ML, U12 INA219AxD, U13 MAX706RESA, U14 INA219AxD, U2 1049, U3 TPS54226PWPRPWP14_2P31X2P46-L, U4 1049, U5 TPS54226PWPRPWP14_2P31X2P46-L, U6 TPS7A4501DCQT, U7 ADS1015IDGS, U8 W25Q128JV, U9 AD8495, Y1 Crystal_GND24, Y2 Crystal_GND24

Commit message: Big Update of In Dev Boards
Mid Term update for all the boards being developed for use by the Irvington Team on Pleiades - Orpheus
Changed lines of the file:
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@@
   (junction (at 59.69 53.34) (diameter 0) (color 0 0 0 0)
   )
+  (junction (at 499.999 147.32) (diameter 0) (color 0 0 0 0)
+  )
   (junction (at 43.1292 367.8174) (diameter 0) (color 0 0 0 0)
   )
@@
   (junction (at 41.91 284.9372) (diameter 0) (color 0 0 0 0)
   )
-  (junction (at 499.2878 143.256) (diameter 0) (color 0 0 0 0)
-  )
   (junction (at 163.7538 300.99) (diameter 0) (color 0 0 0 0)
   )
@@
   )
   (junction (at 251.46 34.29) (diameter 0) (color 0 0 0 0)
-  )
-  (junction (at 499.2878 147.32) (diameter 0) (color 0 0 0 0)
   )
   (junction (at 435.61 36.83) (diameter 0) (color 0 0 0 0)
@@
     (stroke (width 0) (type default))
   )
+  (wire (pts (xy 499.999 143.256) (xy 499.2878 143.256))
+    (stroke (width 0) (type default))
+  )
   (polyline (pts (xy 12.7 110.49) (xy 273.05 110.49))
     (stroke (width 0) (type dash))
@@
     (stroke (width 0) (type default))
   )
+  (wire (pts (xy 499.999 147.32) (xy 501.65 147.32))
+    (stroke (width 0) (type default))
+  )
   (wire (pts (xy 430.53 58.42) (xy 433.07 58.42))
     (stroke (width 0) (type default))
@@
     (stroke (width 0) (type default))
   )
-  (wire (pts (xy 494.2078 147.32) (xy 499.2878 147.32))
+  (wire (pts (xy 494.2078 147.32) (xy 499.999 147.32))
     (stroke (width 0) (type default))
   )
@@
     (stroke (width 0) (type default))
   )
-  (wire (pts (xy 499.2878 147.32) (xy 501.65 147.32))
-    (stroke (width 0) (type default))
-  )
   (wire (pts (xy 125.73 354.33) (xy 125.73 356.87))
     (stroke (width 0) (type default))
@@
     (stroke (width 0) (type default))
   )
-  (wire (pts (xy 499.2878 143.002) (xy 499.2878 143.256))
-    (stroke (width 0) (type default))
-  )
   (wire (pts (xy 313.69 86.36) (xy 327.66 86.36))
     (stroke (width 0) (type default))
@@
   )
   (wire (pts (xy 372.11 142.24) (xy 372.11 146.05))
+    (stroke (width 0) (type default))
+  )
+  (wire (pts (xy 499.999 143.256) (xy 499.999 147.32))
     (stroke (width 0) (type default))
   )
@@
     (stroke (width 0) (type default))
   )
-  (wire (pts (xy 499.2878 143.256) (xy 499.2878 147.32))
-    (stroke (width 0) (type default))
-  )
