File: flat_sat_dev_board/embedded schematics/EPS.kicad_sch (KiCad schematic)
At the start: 204 parts, among them IC2 PCT2075DP,118, IC3 RP2040_QFN56, IC4 LT3652IMSE#PBF, J1 Bypass, J10 Jetson, J11 BM04B-SRSS-TB(LF)(SN), J14 Solar, J15 FC, J16 I2C Multiplexer Breakout, J17 ISS Foot, J18 Screw_Terminal_01x02, J19 BM04B-SRSS-TB(LF)(SN), J2 Heater, J20 CAN1, J21 BM04B-SRSS-TB(LF)(SN), J22 CAN2, J23 Conn_ARM_JTAG_SWD_10, J24 USB_B_Micro, J25 Life Makes Lemonade, J26 BM04B-SRSS-TB(LF)(SN), J27 I2C0 Breakout, J28 Barrel_Jack_Switch, J3 BURN, J4 CHARGE, J5 Foot0, J6 Foot1, J7 Foot2, J8 Foot3, J9 RBF, K1 APAN3109, Q1 IRF7458, Q10 IRLML2803, Q11 NDS8434, Q2 IRF7458, Q3 MBT2222ADW1T1, Q4 MMBT2222AT, Q5 MBT2222ADW1T1, Q6 IRLML2803, Q7 IRLML2803, Q8 NDS8434, Q9 NDS8434, SW1 KMR2, SW2 KMR2, U1 R5460N208AA, U10 TLVH431 DBZ SOT-23, U11 MCP25625-E/ML, U12 INA219AxD, U13 MAX706RESA, U14 INA219AxD, U2 1049, U3 TPS54226PWPRPWP14_2P31X2P46-L, U4 1049, U5 TPS54226PWPRPWP14_2P31X2P46-L, U6 TPS7A4501DCQT, U7 ADS1015IDGS, U8 W25Q128JV, U9 AD8495, Y1 Crystal_GND24, Y2 Crystal_GND24

Commit message: schematic done?
Parts:
- removed C13: 10uF, Capacitor_SMD:C_0603_1608Metric, symbol Device:C_Small
- removed J11: BM04B-SRSS-TB(LF)(SN), Battery Board:JST_BM04B-SRSS-TB(LF)(SN), symbol BM04B-SRSS-TB_LF__SN_:BM04B-SRSS-TB(LF)(SN)
- removed J14: Solar, Battery Board:MOLEX_5040500591, symbol Max_Lib:Connector_Generic_Conn_01x05
- removed J15: FC, Battery Board:MOLEX_5040500591, symbol Max_Lib:Connector_Generic_Conn_01x05
- removed JP1: SolderJumper_3_Open, Jumper:SolderJumper-3_P1.3mm_Open_RoundedPad1.0x1.5mm_NumberLabels, symbol Jumper:SolderJumper_3_Open
- removed R25: 10K, Resistor_SMD:R_0603_1608Metric, symbol Device:R_US
- removed R26: 3.3K, Resistor_SMD:R_0603_1608Metric, symbol Device:R_US
- removed R62, R63, R64, R65: 1M, Resistor_SMD:R_0603_1608Metric, symbol mainboard:RESISTOR0603
- removed U6: TPS7A4501DCQT, Package_TO_SOT_SMD:SOT-223-6, symbol mainboard:TPS7A4501DCQT
- added J23: ~, flat-sat:Burn_Wire, symbol Antenna:Burn_Wire
- added J29: CHARGE, flat-sat:MOLEX_504050-0291, symbol Connector_Generic:Conn_01x02
- J10, J17, J2, J3, J4, J5, J6, J7, J8, J9: footprint Battery Board:MOLEX_504050-0291 -> flat-sat:MOLEX_504050-0291
- J18: footprint Battery Board:ScrewTerminal -> flat-sat:ScrewTerminal
- J19, J21, J26: footprint Battery Board:JST_BM04B-SRSS-TB(LF)(SN) -> flat-sat:JST_BM04B-SRSS-TB(LF)(SN)
- J23: footprint Battery Board:JTAG_2X05_1.27MM_BOX_NOCREAM -> flat-sat:JTAG_2X05_1.27MM_BOX_NOCREAM
- J24: footprint FC_DEV_BOARD:MOLEX_105164-0001 -> flat-sat:MOLEX_105164-0001
- K1: footprint APAN3105:RELAY_APAN3105 -> flat-sat:RELAY_APAN3105
- SW1, SW2: footprint Battery Board:BTN_KMR2_4.6X2.8 -> flat-sat:BTN_KMR2_4.6X2.8
- U2, U4: footprint 1049:1049 -> flat-sat:1049
- renumbered D11 to D8, D12 to D9, J28 to J18
Connections:
- net +9V: now also D9.2; no longer D9.A
- net BURN: now also J23.1 (Power)
- net D+: now also IC3.47 (USB_D+), R54.1; no longer J24.3 (D+), J26.3, R54.2
- net D-: now also IC3.46 (USB_D-), R53.1; no longer J24.2 (D-), J26.2, R53.2
- net FC_RX: now also D3.2; no longer D3.A
- net FC_TX: now also D2.2; no longer D2.A
- net GND: now also D10.1, J23.2 (GND), J29.1 (Pin_1); no longer D10.C
- net USBBOOT: now also D8.1; no longer D8.C
- net USB_D+: now also J24.3 (D+), J26.3, R54.2; no longer IC3.47 (USB_D+), R54.1
- net USB_D-: now also J24.2 (D-), J26.2, R53.2; no longer IC3.46 (USB_D-), R53.1
- net VBATT_SENSE: now also D6.2, D9.2; no longer D6.A, D9.A
- net VBUSP: now also D1.1; no longer D1.C
- net VBatt: now also D9.1, D9.1; no longer D9.C, D9.C
- net VSOLAR: now also J29.2 (Pin_2)
- net at R39.1: now also D2.1; no longer D2.C
- net at K1.C2, Q4.3 (C): now also D1.2; no longer D1.A
- net at C39.2, IC4.11 (BOOST): now also D6.1; no longer D6.C
- net at R57.2: now also D10.2; no longer D10.A
- net at R56.2: now also D8.2; no longer D8.A
- net at R41.1: now also D3.1; no longer D3.C
- net SCL1 renamed EPS_SCL1
- net SDA1 renamed EPS_SDA1
Other:
- note removed: "RF Regulator"
- note removed: "Radio VDD Select"
- note removed: "Set RF Voltage: VOUT=1.21*(1+R55/R59)+(3E-6*R55) VOUT=5V (R55=10K, R59=3.3K)"
- moved on the sheet: C35, C36, C37, C38, C41, C42, C50, D2, D3, D5, IC2, J10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

Commit message: layout on flat-sat board nearly done
Parts:
- removed J22: CAN2, Connector_JST:JST_SH_SM04B-SRSS-TB_1x04-1MP_P1.00mm_Horizontal, symbol Connector_Generic:Conn_01x04
- J30: renamed from J20; footprint Connector_JST:JST_SH_SM04B-SRSS-TB_1x04-1MP_P1.00mm_Horizontal -> Connector_JST:JST_SH_BM04B-SRSS-TB_1x04-1MP_P1.00mm_Vertical
- R40: renamed from R51; value 629k -> 634k
- R43: renamed from R52; value 415k -> 412k
- TP13: renamed from TP8; value TestPoint -> USBBOOT
- renumbered C34 to C46, C39 to C47, C40 to C48, C43 to C49, C44 to C50, C45 to C51, C46 to C52, C47 to C53, C14 to C54, C15 to C55, C5 to C56, C7 to C57, C48 to C58, C8 to C59, C49 to C60, C9 to C61, C50 to C62, C17 to C63, C18 to C64, C19 to C65, C22 to C66, C41 to C67, C42 to C68, C16 to C69, C1 to C70, C2 to C71, C3 to C72, C24 to C73, C4 to C74, C27 to C75, C6 to C76, C20 to C77, C21 to C78, C23 to C79, C25 to C80, C26 to C81, C28 to C82, C38 to C83, C37 to C84, C29 to C85, C30 to C86, C31 to C87, C32 to C88, C10 to C89, C33 to C90, C11 to C91, C12 to C92, C35 to C93, C36 to C94, D6 to D10, D7 to D11, D9 to D12, D10 to D13, D2 to D14, D3 to D15, D8 to D16, D5 to D17, D4 to D6, D1 to D7, FB1 to FB3, FB2 to FB4, FB3 to FB5, IC2 to IC3, IC3 to IC5, J5 to J12, J1 to J13, J17 to J14, J6 to J15, J2 to J16, J7 to J17, J3 to J19, J8 to J20, J4 to J21, J9 to J22, J21 to J24, J10 to J26, J19 to J27, J26 to J28, J16 to J31, J27 to J32, J18 to J34, J23 to J35, J24 to J36, JP2 to JP12, L1 to L4, LED1 to LED2, Q11 to Q10, Q3 to Q11, Q5 to Q12, Q4 to Q2, Q6 to Q3, Q7 to Q4, Q8 to Q5, Q9 to Q6, Q1 to Q7, Q2 to Q8, Q10 to Q9, R58 to R30, R9 to R31, R2 to R32, R60 to R33, R43 to R34, R44 to R35, R47 to R36, R19 to R37, R21 to R38, R22 to R39, R23 to R41, R24 to R42, R27 to R44, R28 to R45, R55 to R46, R1 to R47, R3 to R48, R29 to R49, R30 to R50, R16 to R51, R61 to R52, R59 to R53, R18 to R54, R4 to R55, R20 to R56, R5 to R57, R57 to R58, R32 to R59, R33 to R60, R34 to R61, R53 to R62, R54 to R63, R49 to R64, R50 to R65, R37 to R66, R39 to R67, R41 to R68, R56 to R69, R35 to R70, R45 to R71, R31 to R72, R36 to R73, R38 to R74, R40 to R75, R46 to R76, R42 to R77, R6 to R78, R7 to R79, R8 to R80, R10 to R81, R11 to R82, R12 to R83, R13 to R84, R14 to R85, R15 to R86, R48 to R87, R17 to R88, SW1 to SW3, SW2 to SW4, TP4 to TP10, TP5 to TP11, TP6 to TP12, TP7 to TP14, TP9 to TP6, TP1 to TP7, TP2 to TP8, TP3 to TP9, U2 to U13, U1 to U14, U4 to U15, U5 to U16, U9 to U17, U10 to U18, U12 to U19, U14 to U20, U13 to U21, U7 to U22, U8 to U23, U11 to U24, U3 to U25, Y1 to Y4, Y2 to Y5
Connections:
- net BURN: now also J19.1 (Pin_1); no longer J19.2 (Pin_2)
- net GND: now also J16.2 (Pin_2), J19.2 (Pin_2); no longer J16.1 (Pin_1), J19.1 (Pin_1)
- net Heater: now also J16.1 (Pin_1); no longer J16.2 (Pin_2)
- net VBUSP: now also J22.2 (Pin_2); no longer J22.1 (Pin_1)
- net VBatt: now also J12.1 (Pin_1); no longer J12.2 (Pin_2)
- net VBatt1: now also J15.2 (Pin_2), J22.1 (Pin_1); no longer J15.1 (Pin_1), J22.2 (Pin_2)
- new net: J12.2 (Pin_2), J15.1 (Pin_1)
