File: flat_sat_dev_board/embedded schematics/Flight_Computer.kicad_sch (KiCad schematic)
At the start: 96 parts, among them IC1 RP2040_QFN56, IC2 AZ1117CH-3.3TRG1, J1 Conn_ARM_JTAG_SWD_10, J10 BM04B-SRSS-TB(LF)(SN), J11 BM04B-SRSS-TB(LF)(SN), J12 BM04B-SRSS-TB(LF)(SN), J13 Breakout, J14 Battery, J15 Breakout, J2 FC to EPS Connector, J3 Life Makes Lemonade, J4 104031-0811, J5 BM04B-SRSS-TB(LF)(SN), J6 Conn_Coaxial, J7 Breakout, J8 USB_B_Micro, J9 BM04B-SRSS-TB(LF)(SN), SW1 KMR2, SW2 KMR2, U10 AP3602AKTR-G1, U3 MAX706RESA, U4 RFM98PW, U5 RFM9xBreakout, U6 W25Q128JV, U7 LSM6DSOTR, U8 LSM303AGRTR, U9 MCP25625-E/ML, Y1 12MHZ, Y3 16MHZ 12 pf

Commit message: schematic done?
Parts:
- removed C12: 10uF, Capacitor_SMD:C_0603_1608Metric, symbol Adafruit ItsyBitsy RP2040-eagle-import:CAP_CERAMIC_0603MP
- removed C13: 22uF, Capacitor_SMD:C_0603_1608Metric, symbol Adafruit ItsyBitsy RP2040-eagle-import:CAP_CERAMIC_0603MP
- removed IC2: AZ1117CH-3.3TRG1, Package_TO_SOT_SMD:SOT-223, symbol AZ1117CH-3.3TRG1:AZ1117CH-3.3TRG1
- removed J10, J11, J12: BM04B-SRSS-TB(LF)(SN), FC_DEV_BOARD:JST_BM04B-SRSS-TB(LF)(SN), symbol BM04B-SRSS-TB_LF__SN_:BM04B-SRSS-TB(LF)(SN)
- removed J14: Battery, FC_DEV_BOARD:MOLEX_5040500591, symbol Max_Lib:Connector_Generic_Conn_01x05
- removed J15: Breakout, Connector_JST:JST_SH_BM04B-SRSS-TB_1x04-1MP_P1.00mm_Vertical, symbol Connector_Generic:Conn_01x04
- removed J7: Breakout, Connector_JST:JST_SH_SM04B-SRSS-TB_1x04-1MP_P1.00mm_Horizontal, symbol Connector_Generic:Conn_01x04
- removed JP1: SolderJumper_2_Open, Jumper:SolderJumper-2_P1.3mm_Open_RoundedPad1.0x1.5mm, symbol Jumper:SolderJumper_2_Open
- removed R15: 10k, Resistor_SMD:R_0402_1005Metric, symbol Adafruit ItsyBitsy RP2040-eagle-import:RESISTOR_0402NO
- added C12, C4: 10nf, Capacitor_SMD:C_0402_1005Metric, symbol Adafruit ItsyBitsy RP2040-eagle-import:CAP_CERAMIC_0402NO
- added C17, C18, C19, C20, C24, C39: 0.1uF, Capacitor_SMD:C_0603_1608Metric, symbol Adafruit Ethernet FeatherWing-eagle-import:CAP_CERAMIC0603_NO
- added C21, C23, C34: 10uF, Capacitor_SMD:C_0805_2012Metric, symbol Adafruit Ethernet FeatherWing-eagle-import:CAP_CERAMIC0805-NOOUTLINE
- added C3, C6: 6.8nf, Capacitor_SMD:C_0402_1005Metric, symbol Adafruit ItsyBitsy RP2040-eagle-import:CAP_CERAMIC_0402NO
- added C36, C37: 22pF, Capacitor_SMD:C_0402_1005Metric, symbol Adafruit Ethernet FeatherWing-eagle-import:CAP_CERAMIC0603_NO
- added C42, C44: 10uF, Capacitor_SMD:C_0805_2012Metric, symbol Adafruit VL6180 Time of Flight Sensor-eagle-import:CAP_CERAMIC0805-NOOUTLINE
- added C43: 100nf, Capacitor_SMD:C_0603_1608Metric, symbol Device:C
- added C45: 0.1uF, Capacitor_SMD:C_0603_1608Metric, symbol Adafruit VL6180 Time of Flight Sensor-eagle-import:CAP_CERAMIC0603_NO
- added FB1, FB2: FerriteBead, Resistor_SMD:R_0603_1608Metric, symbol Device:FerriteBead
- added IC2: PCT2075DP,118, Package_SO:TSSOP-8_3x3mm_P0.65mm, symbol Antenna:PCT2075DP,118
- added J1: RJ45_LED_Shielded, flat-sat:RB1-125BAG1A_WIZ, symbol Connector:RJ45_LED_Shielded
- added J8: Breakout, Connector_JST:JST_SH_SM04B-SRSS-TB_1x04-1MP_P1.00mm_Horizontal, symbol Connector_Generic:Conn_01x04
- added JP10, JP8, JP9: SolderJumper_2_Open, Jumper:SolderJumper-2_P1.3mm_Open_RoundedPad1.0x1.5mm, symbol Jumper:SolderJumper_2_Open
- added Q1: BSS138, Package_TO_SOT_SMD:SOT-363_SC-70-6, symbol Adafruit VL6180 Time of Flight Sensor-eagle-import:MOSFET-N_DUAL
- added R10, R4, R6, R9: 49.9, Resistor_SMD:R_0603_1608Metric, symbol mainboard:RESISTOR0603
- added R12: 10k, Resistor_SMD:R_0603_1608Metric, symbol mainboard:RESISTOR0603
- added R20: 12.4k, Resistor_SMD:R_0603_1608Metric, symbol mainboard:RESISTOR0603
- added R25: 1M, Resistor_SMD:R_0603_1608Metric, symbol mainboard:RESISTOR0603
- added R26: 10k, Resistor_SMD:R_Array_Convex_4x0603, symbol Device:R_Pack04
- added R27, R28: 10K, Resistor_SMD:R_0603_1608Metric, symbol Adafruit VL6180 Time of Flight Sensor-eagle-import:RESISTOR_0603_NOOUT
- added R29: 10K, Resistor_SMD:R_Array_Convex_4x0603, symbol Adafruit VL6180 Time of Flight Sensor-eagle-import:RESISTOR_4PACK
- added R8: 10, Resistor_SMD:R_0603_1608Metric, symbol mainboard:RESISTOR0603
- added U11: VL6180XV0NR/1, flat-sat:VL6180, symbol VL6180X0NR:VL6180XV0NR/1
- added U12: LP5907-2.8V, Package_TO_SOT_SMD:SOT-23-5, symbol Adafruit VL6180 Time of Flight Sensor-eagle-import:VREG_SOT23-5
- added U3: SN74AHC1G125DBVR, Package_TO_SOT_SMD:SOT-23-5, symbol 74AHC1G125:SN74AHC1G125DBVR
- added U6: W5500, Package_QFP:LQFP-48_7x7mm_P0.5mm, symbol W5500:W5500
- added Y3: 25MHz, Crystal:Crystal_SMD_3225-4Pin_3.2x2.5mm, symbol Adafruit Ethernet FeatherWing-eagle-import:CRYSTAL3.2X2.5
- J1: footprint FC_DEV_BOARD:JTAG_2X05_1.27MM_BOX_NOCREAM -> flat-sat:JTAG_2X05_1.27MM_BOX_NOCREAM
- J5, J9: footprint FC_DEV_BOARD:JST_BM04B-SRSS-TB(LF)(SN) -> flat-sat:JST_BM04B-SRSS-TB(LF)(SN)
- J8: footprint FC_DEV_BOARD:MOLEX_105164-0001 -> flat-sat:MOLEX_105164-0001
- SW1, SW2: footprint FC_DEV_BOARD:BTN_KMR2_4.6X2.8 -> flat-sat:BTN_KMR2_4.6X2.8
- U4: footprint FC_DEV_BOARD:RFM98PW -> flat-sat:RFM98PW
Connections:
- net VCC_RF1 is gone; now on net +5V: JP10.3 (B), JP7.1 (A)
- net +3V3: now also LED1.1 (VDD), C34.1, C39.1, C42.1, C43.1, FB2.1, IC2.8 (VCC), J1.10, J1.12, J8.2 (Pin_2), R12.1, R26.5 (R4.2), R26.6 (R3.2), R26.7 (R2.2), R26.8 (R1.2), R29.1, R29.3 (1), U12.1 (IN), U12.3 (EN), U3.5 (VCC), U6.28 (VDD)
- net GND: now also C34.2, C36.2, C37.2, C39.2, C42.2, C43.2, C44.2, C45.2, FB1.1, IC2.4 (GND), IC2.5 (A2), IC2.6 (A1), IC2.7 (A0), J1.4, J1.5, J8.1 (Pin_1), JP10.1 (A), JP8.1 (A), JP9.1 (A), U11.12 (AVSS), U11.9 (AVSS_VCSEL), U12.2 (GND), U3.3 (GND), U6.23 (RSVD), U6.29 (GND)
- net SCL1: now also IC2.2 (SCL), J8.4 (Pin_4), Q1.6 (D), R29.8 (2)
- net SDA1: now also IC2.1 (SDA), J8.3 (Pin_3), Q1.3 (D), R29.6 (2)
- net SPI0_CS1: now also R12.2
- net SPI0_MISO: now also U3.4 (Y)
- net SPI0_MOSI: now also U6.35 (MOSI)
- net SPI0_SCK: now also U6.33 (SCLK)
- net Neo_pwr renamed SPI0_CS3
- net SPI0_CS3: now also U3.1 (*OE), U6.32 (SCSN); no longer LED1.1 (VDD)
- net RX renamed FC_RX
- net SCL0 renamed FC_SCL0
- net SDA0 renamed FC_SDA0
- net TX renamed FC_TX
- net VBUS renamed FC_USB_pwr
- new net: C3.1, J1.7
- new net: JP8.2 (B), R26.1 (R1.1), U6.45 (PMODE0)
- new net: JP9.2 (B), R26.2 (R2.1), U6.44 (PMODE1)
- new net: JP10.2 (B), R26.3 (R3.1), U6.43 (PMODE2)
- new net: R26.4 (R4.1), U6.36 (INTN)
- new net: R20.2, U6.10 (EXRES1)
- new net: C37.1, R25.1, U6.30 (XI/CLKIN), Y3.1
- new net: C36.1, R25.2, U6.31 (XO), Y3.3 (2)
- new net: C6.1, J1.8
- new net: C24.2, U6.22 (1V20)
- new net: C23.2, U6.20 (TOCAP)
- new net 2.8V: C44.1, C45.1, Q1.2 (G), Q1.5 (G), R27.2, R28.2, R29.2 (1), R29.4 (1), U11.10 (AVDD), U11.8 (AVDD_VCSEL), U12.5 (OUT)
- new net GNDA: C12.2, C17.2, C18.2, C19.2, C20.2, C21.2, C23.1, C24.1, C4.2, FB1.2, R20.1, U6.14 (AGND), U6.16 (AGND), U6.19 (AGND), U6.3 (AGND), U6.48 (AGND), U6.9 (AGND)
- new net GPIO: R27.1, U11.1 (GPIO1)
- new net GREENLED: J1.9, U6.25 (LINKLED)
- new net MISO_ETHER: U3.2 (A), U6.34 (MISO)
- new net RCT: C4.1, J1.6, R4.2, R6.2
- new net RX+: C3.2, R4.1, U6.6 (RXP)
- new net RX-: C6.2, R6.1, U6.5 (RXN)
- new net SCL_3V: Q1.1 (S), R29.7 (2), U11.5 (SCL)
- new net SDA_3V: Q1.4 (S), R29.5 (2), U11.6 (SDA)
- new net TCT: C12.1, J1.3, R8.2
- new net TX+: J1.1, R10.2, U6.2 (TXP)
- new net TX-: J1.2, R9.2, U6.1 (TXN)
- new net VDDA: C17.1, C18.1, C19.1, C20.1, C21.1, FB2.2, R10.1, R8.1, R9.1, U6.11 (AVDD), U6.15 (AVDD), U6.17 (AVDD), U6.21 (AVDD), U6.4 (AVDD), U6.8 (AVDD)
- new net XSHUT_2.8V: R28.1, U11.4 (GPIO0)
- new net YELLOWLED: J1.11, U6.27 (ACTLED)
- no-connect marks 33 -> 43
Other:
- note added: "0 0 0 = 10BT Half-duplex, Auto-negotiation disabled 0 0 1 = 10BT Full-duplex, Auto-negotiation disabled 0 1 0 = 100BT Half-duplex, Auto-negotiation disabled 0 1 1 = 100BT Full-duplex, Auto-negotiation disabled 1 0 0 = 100BT Half-duplex, Auto-negotiation enabled 1 1 1 = All capable, Auto-negotiation enabled (DEFAULT)"
- note added: "D"
- note added: "G"
- note added: "S"
- note removed: "3v3 Linear Regulator"
- note removed: "For USB Power"
- moved on the sheet: C34, C35, C39, C40, D1, D2, J13, J3, J5, JP10, JP4, R24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

Commit message: layout on flat-sat board nearly done
Parts:
- removed C41: 10uf, Capacitor_SMD:C_0603_1608Metric, symbol Adafruit Ethernet FeatherWing-eagle-import:CAP_CERAMIC0603_NO
- removed C42: 1uf, Capacitor_SMD:C_0603_1608Metric, symbol Adafruit Ethernet FeatherWing-eagle-import:CAP_CERAMIC0603_NO
- removed R27: 10k, Resistor_SMD:R_0603_1608Metric, symbol mainboard:10KOHM-1_10W-1%(0603)0603
- removed TP5: 5V, TestPoint:TestPoint_Loop_D1.80mm_Drill1.0mm_Beaded, symbol Connector:TestPoint
- removed U10: AP3602AKTR-G1, Package_TO_SOT_SMD:SOT-23-6, symbol AP3602:AP3602AKTR-G1
- renumbered C7 to C10, C8 to C11, C9 to C13, C10 to C14, C11 to C15, C35 to C16, C34 to C22, C38 to C25, C37 to C26, C32 to C27, C31 to C28, C14 to C29, C40 to C30, C39 to C31, C43 to C32, C15 to C33, C16 to C35, C33 to C41, C3 to C5, C4 to C7, C5 to C8, C6 to C9, D4 to D1, D3 to D2, D2 to D3, D1 to D4, D8 to D5, J13 to J10, J6 to J11, J3 to J2, J1 to J3, J9 to J5, J8 to J6, J5 to J7, J2 to J9, JP4 to JP1, JP10 to JP11, JP9 to JP2, JP8 to JP3, JP5 to JP4, JP7 to JP5, JP3 to JP6, JP6 to JP7, R10 to R1, R6 to R11, R9 to R13, R3 to R14, R4 to R15, R7 to R16, R8 to R17, R24 to R18, R23 to R19, R1 to R2, R25 to R21, R13 to R22, R26 to R24, R2 to R3, R12 to R7, U6 to U1, U5 to U10, U3 to U2, U7 to U4, U9 to U5, U8 to U7, U4 to U9, Y3 to Y2
