File: flat_sat_dev_board/embedded schematics/payload.kicad_sch (KiCad schematic)
At the start: 47 parts, among them IC1 PCA9685PW,118, U1 TCA9548APWR, U1 VEML7700, U15 VEML7700, U16 DRV2605LDGS, U17 MCP9808_DFN, U18 VEML7700, U19 DRV2605LDGS, U2 DRV2605LDGS, U20 MCP9808_DFN, U21 VEML7700, U22 DRV2605LDGS, U23 MCP9808_DFN, U24 VEML7700, U25 DRV2605LDGS, U26 MCP9808_DFN, U3 MCP9808_DFN

Commit message: schematic done?
Parts:
- removed U5: ~, camera_daughter:camera_daughter, symbol camera_daughter:camera_daughter
- added U39: ~, flat-sat:camera_daughter, symbol camera_daughter:camera_daughter
- IC1: footprint PCA9685:SOP65P640X110-28N -> Package_SO:TSSOP-28_8x9.7mm_P0.65mm
- U1: footprint VEML7700-TT:XDCR_VEML7700-TT -> flat-sat:XDCR_VEML7700-TT
- U1: footprint TCA9548APWR:SOP65P640X120-24N -> Package_SO:TSSOP-24_6.1x7.8mm_P0.65mm
- U29: renamed from U15; footprint VEML7700-TT:XDCR_VEML7700-TT -> flat-sat:XDCR_VEML7700-TT
- U33: renamed from U18; footprint VEML7700-TT:XDCR_VEML7700-TT -> flat-sat:XDCR_VEML7700-TT
- U36: renamed from U21; footprint VEML7700-TT:XDCR_VEML7700-TT -> flat-sat:XDCR_VEML7700-TT
- U40: renamed from U24; footprint VEML7700-TT:XDCR_VEML7700-TT -> flat-sat:XDCR_VEML7700-TT
- renumbered C38 to C100, C51 to C101, C52 to C102, C53 to C103, C54 to C104, C55 to C105, C56 to C106, C57 to C107, C58 to C108, C59 to C109, C36 to C98, C37 to C99, D13 to D19, D14 to D20, D15 to D21, D16 to D22, R66 to R91, R67 to R95, R68 to R96, R69 to R97, U16 to U30, U17 to U31, U20 to U34, U19 to U35, U22 to U37, U23 to U38, U25 to U41, U26 to U42
Connections:
- net +3V3: now also U39.5 (Pwr)
- net GND: now also U39.1 (GND)
- net Camera renamed payload
- net payload: now also U39.2 (ps)
- net SCL0 renamed FC_SCL0
- net FC_SCL0: now also U39.4 (SCL)
- net SCL1 renamed EPS_SCL1
- net SDA0 renamed FC_SDA0
- net FC_SDA0: now also U39.3 (SDA)
- net SDA1 renamed EPS_SDA1
Other:
- moved on the sheet: C101, C102, C103, C104, C105, C106, C107, C108, C109, D20, D21, D22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

Commit message: layout on flat-sat board nearly done
Parts:
- added J33: Driver0, flat-sat:MOLEX_504050-0291, symbol Connector_Generic:Conn_01x02
- added J37: Driver1, flat-sat:MOLEX_504050-0291, symbol Connector_Generic:Conn_01x02
- added J38: Driver2, flat-sat:MOLEX_504050-0291, symbol Connector_Generic:Conn_01x02
- added J39: Driver3, flat-sat:MOLEX_504050-0291, symbol Connector_Generic:Conn_01x02
- added J40: Driver4, flat-sat:MOLEX_504050-0291, symbol Connector_Generic:Conn_01x02
- renumbered C1 to C95, C2 to C96, C3 to C97, D4 to D18, IC1 to IC6, R1 to R89, R1 to R90, R2 to R92, R3 to R93, R4 to R94, U1 to U26, U2 to U27, U3 to U28, U1 to U32
Connections:
- net at U30.7 (OUT+): now also J37.1 (Pin_1); no longer U30.9 (OUT-)
- net at U27.7 (OUT+): now also J33.1 (Pin_1); no longer U27.9 (OUT-)
- net at U35.7 (OUT+): now also J38.1 (Pin_1); no longer U35.9 (OUT-)
- net at U41.7 (OUT+): now also J40.1 (Pin_1); no longer U41.9 (OUT-)
- net at U37.7 (OUT+): now also J39.1 (Pin_1); no longer U37.9 (OUT-)
- new net: J40.2 (Pin_2), U41.9 (OUT-)
- new net: J37.2 (Pin_2), U30.9 (OUT-)
- new net: J33.2 (Pin_2), U27.9 (OUT-)
- new net: J38.2 (Pin_2), U35.9 (OUT-)
- new net: J39.2 (Pin_2), U37.9 (OUT-)
