File: Z_Face/solar-panel-side-Z.kicad_sch (KiCad schematic)
At the start: 30 parts, among them J1 CON-5040500591, J10 Face0, J11 Face1, J12 Face2, J13 Face3, J4 Conn_01x01, J5 Conn_01x01, J6 Conn_01x01, J7 Conn_01x01, U1 VEML7700, U2 DRV2605LDGS, U3 MCP9808_DFN

Commit message: Big Update of In Dev Boards
Mid Term update for all the boards being developed for use by the Irvington Team on Pleiades - Orpheus
Parts:
- U3: footprint SolarPanelBoards:MCP9808-NoLeadPackage -> Package_SO:MSOP-8-1EP_3x3mm_P0.65mm_EP2.5x3mm_Mask1.73x2.36mm
- U5: footprint (none) -> camera_daughter:camera_daughter
Changed lines of the file:
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@@
       (effects (font (size 1.27 1.27)))
     )
-    (property "Footprint" "" (at 161.5694 51.7906 0)
+    (property "Footprint" "camera_daughter:camera_daughter" (at 161.5694 51.7906 0)
       (effects (font (size 1.27 1.27)) hide)
     )
@@
       (effects (font (size 1.27 1.27)) (justify left))
     )
-    (property "Footprint" "SolarPanelBoards:MCP9808-NoLeadPackage" (at 45.72 92.71 0)
-      (effects (font (size 1.27 1.27)) hide)
-    )
+    (property "Footprint" "Package_SO:MSOP-8-1EP_3x3mm_P0.65mm_EP2.5x3mm_Mask1.73x2.36mm" (at 45.72 92.71 0)
+      (effects (font (size 1.27 1.27)) hide)
+    )

Commit message: schematic done?
Connections:
- net 3v3_break: now also U5.5 (Pwr)
- net Camera_Pwr renamed Camera_Pwr_select

Commit message: Squashed commit of the following:
commit e254adcde77272bf9c297392939bbb8f65e8d1c6
Author: Michael Pham <61564344+Mikefly123@users.noreply.github.com>
Date:   Tue May 28 21:23:36 2024 -0700

    Fixed Antenna Board

commit 045481aa1d64479ef8ca8c2eedf132e30a3c2c12
Author: Michael Pham <61564344+Mikefly123@users.noreply.github.com>
Date:   Tue May 28 20:29:56 2024 -0700

    Consolidating files

commit 0d9b312b1d72281e33c094203cb00ac56d2c935d
Author: kdizzlle <112121179+kdizzlle@users.noreply.github.com>
Date:   Tue May 28 13:55:35 2024 -0700

    added extra pin to z face

    moved it slightly closer also
Connections:
- net +3V3: now also U5.5 (3V3)
- net 3v3_break: no longer U5.5 (Pwr)
- net Camera_Pwr_select renamed Camera_Pwr
