File: sx1276-dev/radio_module.kicad_sch (KiCad schematic)
At the start: 62 parts, among them J1 Conn_Coaxial, J2 Conn_Coaxial, U1 SX1276, U2 4259-63, U3 4259-63, Y1 32.0MHz

Commit message: Updated Schematic
Parts:
- removed C1, C2: 15pF, symbol Device:C
- removed C12, C15, C33, C34, C37: C, symbol Device:C
- removed C38: 10nF, symbol Device:C
- removed C4, C7, C8: 100nF, symbol Device:C
- removed C40: 47nF, symbol Device:C
- removed L11, L12, L4, L9: L, symbol Device:L
- removed U1: SX1276, Package_DFN_QFN:QFN-28-1EP_6x6mm_P0.65mm_EP4.8x4.8mm, symbol RF:SX1276
- removed Y1: 32.0MHz, symbol Device:Crystal_GND24
- added C1, C52: 1u, Capacitor_SMD:C_0402_1005Metric, symbol Device:C_Small
- added C10, C43: 0.1uF, Capacitor_SMD:C_0402_1005Metric, symbol Device:C
- added C13, C48: 100pF, Capacitor_SMD:C_0402_1005Metric, symbol Device:C
- added C18, C47: 12pf, Capacitor_SMD:C_0402_1005Metric, symbol Device:C
- added C2, C4, C53, C55: 100p, Capacitor_SMD:C_0402_1005Metric, symbol Device:C_Small
- added C21: 15pF, Capacitor_SMD:C_0402_1005Metric, symbol Device:C
- added C23, C24, C32: 100nF, Capacitor_SMD:C_0402_1005Metric, symbol Device:C
- added C25: 1nF, Capacitor_SMD:C_0402_1005Metric, symbol Device:C
- added C27: 10nF, Capacitor_SMD:C_0402_1005Metric, symbol Device:C
- added C28, C29: 47nF, Capacitor_SMD:C_0402_1005Metric, symbol Device:C
- added C44: 22uF, Capacitor_SMD:C_0603_1608Metric, symbol Device:C
- added C45, C46: 1uF, Capacitor_SMD:C_0402_1005Metric, symbol Device:C
- added C49: 5.6pF, Capacitor_SMD:C_0402_1005Metric, symbol Device:C
- added C50: 18pF, Capacitor_SMD:C_0402_1005Metric, symbol Device:C
- added C51: 6.2pF, Capacitor_SMD:C_0402_1005Metric, symbol Device:C
- added C54: 100p, Capacitor_SMD:C_0402_1005Metric, symbol Device:C
- added FB1: FerriteBead, Inductor_SMD:L_0402_1005Metric, symbol Device:FerriteBead
- added IC1, IC2: GRF5112, GRF5112:QFN50P300X300X90-17N, symbol GRF5112:GRF5112
- added J3, J4: Conn_01x08_Socket, symbol Connector:Conn_01x08_Socket
- added L1, L18: 68n, Inductor_SMD:L_0603_1608Metric, symbol Device:L_Small
- added L14, L15: 3.3nH, Inductor_SMD:L_0402_1005Metric, symbol Device:L
- added L16: 3.9nH, Inductor_SMD:L_0402_1005Metric, symbol Device:L
- added L17: 2.4nH, Inductor_SMD:L_0402_1005Metric, symbol Device:L
- added L7: 22nH, Inductor_SMD:L_0402_1005Metric, symbol Device:L
- added L8: 18nH, Inductor_SMD:L_0402_1005Metric, symbol Device:L
- added R10, R3, R5, R9: 0, Resistor_SMD:R_0402_1005Metric, symbol Device:R
- added R11, R13, R14, R16, R17, R18, R19, R21, R22, R23, R24, R25: 100, Resistor_SMD:R_0402_1005Metric, symbol Device:R
- added R12: 4.75k, Resistor_SMD:R_0402_1005Metric, symbol Device:R
- added R15, R7: 50, Resistor_SMD:R_0402_1005Metric, symbol Device:R
- added R20, R6: 15k, Resistor_SMD:R_0402_1005Metric, symbol Device:R
- added R4: 6k, Resistor_SMD:R_0402_1005Metric, symbol Device:R
- added R8: 1k, Resistor_SMD:R_0402_1005Metric, symbol Device:R
- added U1, U6: TQP3M9036, ul_TQP3M9036:DFN8_2x2_QOR, symbol ul_TQP3M9036:TQP3M9036
- added U3: NC7SZ04P5X, NC7SZ04:SC-88A-5_1P35X2P2_ONS, symbol NC7SZ04:NC7SZ04P5X
- added U4: SX1276IMLTRT, SX1276IMLTRT:QFN28_6X6_SEM, symbol SX1276IMLTRT:SX1276IMLTRT
- added XTAL1: NX2016SA-32M-EXS00A-CS06465, NX2016SA_32M_EXS00A_CS06465:NX2016SA_NDK, symbol NX2016SA-32M-EXS00A-CS06465:NX2016SA-32M-EXS00A-CS06465
- C11: renamed from C29; footprint (none) -> Capacitor_SMD:C_0402_1005Metric
- C12: renamed from C11; footprint (none) -> Capacitor_SMD:C_0402_1005Metric
- C14: renamed from C10; value C -> 15nF; footprint (none) -> Capacitor_SMD:C_0402_1005Metric
- C15: renamed from C9; footprint (none) -> Capacitor_SMD:C_0402_1005Metric
- C16: renamed from C13; footprint (none) -> Capacitor_SMD:C_0402_1005Metric
- C17: renamed from C14; footprint (none) -> Capacitor_SMD:C_0402_1005Metric
- C19: value C -> 100pF; footprint (none) -> Capacitor_SMD:C_0402_1005Metric
- C20: value C -> 12pF; footprint (none) -> Capacitor_SMD:C_0402_1005Metric
- C22: value C -> 1pF; footprint (none) -> Capacitor_SMD:C_0402_1005Metric
- C26, C30: value C -> 100nF; footprint (none) -> Capacitor_SMD:C_0402_1005Metric
- C3: value 100nF -> 100p; footprint (none) -> Capacitor_SMD:C_0402_1005Metric
- C31: value C -> 47pF; footprint (none) -> Capacitor_SMD:C_0402_1005Metric
- C33: renamed from C17; footprint (none) -> Capacitor_SMD:C_0402_1005Metric
- C34: renamed from C27; footprint (none) -> Capacitor_SMD:C_0402_1005Metric
- C35: renamed from C16; footprint (none) -> Capacitor_SMD:C_0402_1005Metric
- C36: renamed from C18; footprint (none) -> Capacitor_SMD:C_0402_1005Metric
- C37: renamed from C21; footprint (none) -> Capacitor_SMD:C_0402_1005Metric
- C38: renamed from C32; footprint (none) -> Capacitor_SMD:C_0402_1005Metric
- C39: value 47nF -> 100nF; footprint (none) -> Capacitor_SMD:C_0402_1005Metric
- C40: renamed from C24; footprint (none) -> Capacitor_SMD:C_0402_1005Metric
- C41: renamed from C25; footprint (none) -> Capacitor_SMD:C_0402_1005Metric
- C42: renamed from C23; footprint (none) -> Capacitor_SMD:C_0402_1005Metric
- C5: value 47pF -> 15pF; footprint (none) -> Capacitor_SMD:C_0402_1005Metric
- C6: value 100nF -> 15pF; footprint (none) -> Capacitor_SMD:C_0402_1005Metric
- C7: renamed from C35; footprint (none) -> Capacitor_SMD:C_0402_1005Metric
- C8: renamed from C36; footprint (none) -> Capacitor_SMD:C_0402_1005Metric
- C9: renamed from C28; footprint (none) -> Capacitor_SMD:C_0402_1005Metric
- L10: renamed from L6; footprint (none) -> Inductor_SMD:L_0402_1005Metric
- L11: renamed from L7; footprint (none) -> Inductor_SMD:L_0402_1005Metric
- L12: renamed from L8; footprint (none) -> Inductor_SMD:L_0402_1005Metric
- L13: renamed from L10; footprint (none) -> Inductor_SMD:L_0402_1005Metric
- L2: renamed from L13; footprint (none) -> Inductor_SMD:L_0402_1005Metric
- L3: renamed from L14; footprint (none) -> Inductor_SMD:L_0402_1005Metric
- L4: renamed from L2; footprint (none) -> Inductor_SMD:L_0402_1005Metric
- L5: renamed from L3; footprint (none) -> Inductor_SMD:L_0402_1005Metric
- L6: renamed from L1; value L -> 82nH; footprint (none) -> Inductor_SMD:L_0402_1005Metric
- L9: renamed from L5; footprint (none) -> Inductor_SMD:L_0402_1005Metric
- R1: value R -> 50; footprint (none) -> Resistor_SMD:R_0402_1005Metric
- R2: value 0R -> 0; footprint (none) -> Resistor_SMD:R_0402_1005Metric
- U2: footprint SC-70-6_PSM -> PE4259:SC-70-6_PSM
- U5: renamed from U3; footprint SC-70-6_PSM -> PE4259:SC-70-6_PSM
Connections:
- net +3V3: now also C31.1, C39.1, C23.1, C32.2, C44.1, C45.1, FB1.1, J4.1 (Pin_1), U4.14 (VBAT_DIG), U4.24 (VBAT_RF), U4.3 (VBAT_ANA); no longer C3.1, C34.1, C5.1, C6.1, C9.1, U2.6 (*CTRL/VDD), U5.6 (*CTRL/VDD)
- net DIO0: now also J3.6 (Pin_6), R13.2
- net DIO1: now also J3.7 (Pin_7), R16.2
- net DIO2: now also J3.8 (Pin_8), R18.2
- net DIO3: now also J3.3 (Pin_3), R21.2
- net DIO4: now also J3.4 (Pin_4), R23.2
- net DIO5: now also J4.7 (Pin_7), R24.2
- net GND: now also C20.2, C31.2, R1.1, C1.2, C10.2, C13.2, C2.2, C21.2, C23.2, C24.2, C25.2, C27.2, C28.2, C29.2, C32.1, C43.2, C44.2, C45.2, C46.2, C49.2, C50.2, C51.2, C52.2, C53.2, IC1.11 (GND/NC_6), IC1.13 (GND/NC_7), IC1.15 (GND/NC_8), IC1.16 (GND/NC_9), IC1.17 (GND), IC1.2 (GND/NC_1), IC1.5 (GND/NC_2), IC1.6 (GND/NC_3), IC1.7 (GND/NC_4), IC1.8 (GND/NC_5), IC2.11 (GND/NC_6), IC2.13 (GND/NC_7), IC2.15 (GND/NC_8), IC2.16 (GND/NC_9), IC2.17 (GND), IC2.2 (GND/NC_1), IC2.5 (GND/NC_2), IC2.6 (GND/NC_3), IC2.7 (GND/NC_4), IC2.8 (GND/NC_5), J3.2 (Pin_2), J4.8 (Pin_8), L17.1, L8.1, R20.2, R6.2, R7.1, U1.9 (RF/DC_GND), U3.3 (GND), U4.15 (GND), U4.23 (GND), U4.26 (GND), U4.29 (GND), U6.9 (RF/DC_GND), XTAL1.2, XTAL1.4; no longer C3.2, C31.1
- net MISO: now also J4.2 (Pin_2), R22.2
- net MOSI: now also J4.3 (Pin_3), R19.2
- net NSS: now also J4.5 (Pin_5), R17.2
- net PA_BOOST: now also C49.1, L15.1, U4.27 (PA_BOOST); no longer L10.2
- net RFI_HF: now also U4.21 (RFI_HF); no longer C26.2
- net RFI_LF: now also U4.1 (RFI_LF)
- net RFO_LF: now also C18.1, L8.2, U4.28 (RFO_LF); no longer C14.1, C15.1, L6.2
- net SCK: now also J4.4 (Pin_4), R25.2
- net XTA: now also C5.1, U4.5 (XTA), XTAL1.1
- net XTB: now also C6.1, U4.6 (XTB), XTAL1.3
- net at C38.1: now also J2.1 (In)
- net at C20.1, C22.1: now also C19.1, C21.1, IC1.10 (RF_OUT/VDD_2), IC1.9 (RF_OUT/VDD_1), L7.1; no longer U5.1 (RF1)
- net at C37.1, L12.2: now also U5.1 (RF1); no longer C19.1, C20.2
- net RFI_HF_LNA_IN: now reaches U5.3 (RF2)
- net RFI_HF_LNA_IN: now also C54.1; no longer C41.2
- net RF_CONTROL_SW: now reaches U5.4 (CTRL)
- net RF_CONTROL_SW: now also R11.2, U3.2 (A)
- net at C11.2: now also J1.1 (In); no longer C30.2
- net VR_PA: now reaches L6.1, L9.2
- net VR_PA: now also C27.1, C28.1, C29.1, U4.25 (VR_PA); no longer C39.1
- net at C7.2: now also C8.1; no longer R2.1
- net at C40.2: now also C41.1; no longer R1.1
- net at R1.2: now also R3.1; no longer C41.1
- net at C36.2, L11.2, L12.1: no longer C19.2
- net at C12.1, C16.2, L4.1: now also C14.2
- net at R2.2: now also C10.1, C13.1, L7.2, R5.2; no longer C8.1
- net RFI_LF_LNA_IN: now reaches U2.1 (RF1)
- net RFI_LF_LNA_IN: now also C3.1; no longer C8.2
- net at U2.4 (CTRL): now also C25.1, U3.4 (Y)
- new net: C18.2, IC1.3 (RF_IN_1), IC1.4 (RF_IN_2), R6.1
- new net: C26.2, U4.2 (VR_ANA)
- new net: IC1.1 (VEN1), R4.2
- new net: C43.1, L14.2, R15.2, R9.2
- new net: C50.1, IC2.10 (RF_OUT/VDD_2), IC2.9 (RF_OUT/VDD_1), L14.1, L16.1
- new net: C47.1, L15.2, L17.2
- new net: C47.2, IC2.3 (RF_IN_1), IC2.4 (RF_IN_2), R20.1
- new net: C54.2, U6.2 (RF_IN)
- new net: C30.2, U4.4 (VR_DIG)
- new net: IC1.12 (BIAS2), R5.1
- new net: IC1.14 (BIAS1), R3.2
- new net: IC2.1 (VEN1), R12.2
- new net: C4.2, L1.2, U1.7 (RF_OUT)
- new net: C55.2, L18.2, U6.7 (RF_OUT)
- new net: R10.1, R7.2
- new net: IC2.14 (BIAS1), R10.2
- new net: C48.1, C51.1, L16.2
- new net: IC2.12 (BIAS2), R15.1
- new net: C3.2, U1.2 (RF_IN)
- new net +3.3VA: C1.1, C2.1, C24.1, C34.1, C46.1, C52.1, C53.1, C9.1, FB1.2, L1.1, L18.1, R8.1, U2.6 (*CTRL/VDD), U3.5 (VCC), U5.6 (*CTRL/VDD)
- new net +5V: J3.5 (Pin_5), R12.1, R2.1, R4.1, R9.1
- new net ANT: J3.1 (Pin_1)
- new net DIO0_sx: R13.1, U4.8 (DIO0)
- new net DIO1_sx: R16.1, U4.9 (DIO1)
- new net DIO2_sx: R18.1, U4.10 (DIO2)
- new net DIO3_sx: R21.1, U4.11 (DIO3)
- new net DIO4_sx: R23.1, U4.12 (DIO4)
- new net DIO5_sx: R24.1, U4.13 (DIO5)
- new net HF_PA_OUT: C48.2, L10.2
- new net LF_PA_OUT: C14.1, C15.1, C19.2, L6.2
- new net MISO_sx: R22.1, U4.17 (MISO)
- new net MOSI_sx: R19.1, U4.18 (MOSI)
- new net NRESET: J4.6 (Pin_6), R14.2
- new net NRESET_sx: R14.1, U4.7 (NRESET)
- new net NSS_sx: R17.1, U4.19 (NSS)
- new net RFI_HF_LNA_OUT: C41.2, C55.1
- new net RFI_LF_LNA_OUT: C4.1, C8.2
- new net RF_CONTROL: R11.1, R8.2, U4.20 (RXTX/RFMOD)
- new net SCK_sx: R25.1, U4.16 (SCK)
- no-connect marks 1 -> 3
Other:
- note added: "0402"
- note added: "0603"
- note added: "Crystal"
- note added: "Filtering/Matching Network"
- note added: "LNA HF"
- note added: "LNA LF"
- note added: "PA 433MHz"
- note added: "PA 915MHz"
- note added: "sx1276 Transceiver IC"
- note removed: "20dBm Power amp"
- note removed: "32 MHz crystal"
- note removed: "Crystal, may use TCXO, need to make footprint"
- moved on the sheet: C11, C12, C14, C15, C16, C17, C33, C34, C35, C36, C37, C38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
