File: sx1276-dev/radio_module.kicad_sch (KiCad schematic)
At the start: 112 parts, among them IC1 GRF5112, IC2 GRF5112, J1 Conn_Coaxial, J2 Conn_Coaxial, J3 Conn_01x08_Socket, J4 Conn_01x08_Socket, U1 TQP3M9036, U2 4259-63, U3 NC7SZ04P5X, U4 SX1276IMLTRT, U5 4259-63, U6 TQP3M9036

Commit message: Started Rough Layout
Parts:
- J1, J2: footprint (none) -> Connector_Coaxial:SMA_Amphenol_901-144_Vertical
- J3, J4: footprint (none) -> Connector_PinSocket_1.00mm:PinSocket_1x08_P1.00mm_Vertical
Changed lines of the file:
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@@
 			)
 		)
-		(property "Footprint" ""
+		(property "Footprint" "Connector_PinSocket_1.00mm:PinSocket_1x08_P1.00mm_Vertical"
 			(at 116.84 402.59 0)
 			(effects
@@
 			)
 		)
-		(property "Footprint" ""
+		(property "Footprint" "Connector_Coaxial:SMA_Amphenol_901-144_Vertical"
 			(at 750.57 260.35 0)
 			(effects
@@
 			)
 		)
-		(property "Footprint" ""
+		(property "Footprint" "Connector_PinSocket_1.00mm:PinSocket_1x08_P1.00mm_Vertical"
 			(at 143.51 403.86 0)
 			(effects
@@
 			)
 		)
-		(property "Footprint" ""
+		(property "Footprint" "Connector_Coaxial:SMA_Amphenol_901-144_Vertical"
 			(at 745.49 177.8 0)
 			(effects

Commit message: Updated Schematic and continued layout
Connections:
- net HF_PA_OUT: now also L10.1; no longer L10.2
- net at C33.1, C35.1, L9.1: now also L10.2; no longer L10.1
- net RF_HF_SW: now reaches C37.1, L12.2, U5.1 (RF1)
- net RF_LF_SW: now reaches L5.2, U2.3 (RF2)
Other:
- note added: "Decoupling caps RF choke, and HF bypass caps"
- note added: "Inverter"
- note added: "RF Switch"
- note added: "RF Switch 433MHz"
- note added: "RF Switch 915MHz"
- note added: "Rx 433MHz"
- note added: "Rx 433MHz Filtering/Matching Network"
- note added: "Rx 915MHz Filtering/Matching Network"
- note added: "Rx 915Mhz"
- note added: "Tx 433MHz"
- note added: "Tx 433MHz Filtering/Matching Network"
- note added: "Tx 915MHz Filtering/Matching Network"
- note added: "Tx 915Mhz"
- note added: "VR_PA Circuitry"
- note removed: "Filtering/Matching Network"
- moved on the sheet: C1, C10, C11, C12, C13, C14, C15, C16, C17, C18, C19, C2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

Commit message: Made adjustments to layout
Other:
- note added: "RF Switch 433MHz and SMA Connector"
- note added: "RF Switch 915MHz and SMA connector"
- note removed: "RF Switch 433MHz"
- note removed: "RF Switch 915MHz"
Changed lines of the file:
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@@
 		)
 	)
-	(text "RF Switch 433MHz"
+	(text "RF Switch 433MHz and SMA Connector\n"
 		(exclude_from_sim no)
-		(at 700.024 89.916 0)
+		(at 723.138 88.646 0)
 		(effects
 			(font
@@
 		)
 	)
-	(text "RF Switch 915MHz"
+	(text "RF Switch 915MHz and SMA connector"
 		(exclude_from_sim no)
-		(at 708.406 378.206 0)
+		(at 725.932 376.682 0)
 		(effects
 			(font

Commit message: Added routing to pcb
Parts:
- removed C44: 22uF, Capacitor_SMD:C_0603_1608Metric, symbol Device:C
- removed C45, C46: 1uF, Capacitor_SMD:C_0402_1005Metric, symbol Device:C
- removed FB1: FerriteBead, Inductor_SMD:L_0402_1005Metric, symbol Device:FerriteBead
- J3, J4: value Conn_01x08_Socket -> Conn_01x09_Pin; footprint Connector_PinSocket_1.00mm:PinSocket_1x08_P1.00mm_Vertical -> Connector_PinSocket_1.00mm:PinSocket_1x09_P1.00mm_Vertical; symbol Connector:Conn_01x08_Socket -> Connector:Conn_01x09_Pin
Connections:
- net +3.3VA is gone; now on net +3V3: C1.1, C2.1, C24.1, C34.1, C52.1, C53.1, C9.1, L1.1, L18.1, R8.1, U2.6 (*CTRL/VDD), U3.5 (VCC), U5.6 (*CTRL/VDD)
- net ANT is gone; now on net ANT1: J3.1 (Pin_1)
- net DIO0: now also J3.3 (Pin_3); no longer J3.6 (Pin_6)
- net DIO1: now also J3.4 (Pin_4); no longer J3.7 (Pin_7)
- net DIO2: now also J3.6 (Pin_6); no longer J3.8 (Pin_8)
- net DIO3: now also J3.7 (Pin_7); no longer J3.3 (Pin_3)
- net DIO4: now also J3.8 (Pin_8); no longer J3.4 (Pin_4)
- net DIO5: now also J4.3 (Pin_3); no longer J4.7 (Pin_7)
- net GND: now also J4.9 (Pin_9)
- net MISO: now also J4.5 (Pin_5); no longer J4.2 (Pin_2)
- net MOSI: now also J4.6 (Pin_6); no longer J4.3 (Pin_3)
- net NRESET: now also J4.2 (Pin_2); no longer J4.6 (Pin_6)
- net NSS: now also J4.7 (Pin_7); no longer J4.5 (Pin_5)
- net ANT2: now reaches C38.1, J2.1 (In)
- net ANT2: now also J3.9 (Pin_9)
- net ANT1: now reaches C11.2, J1.1 (In)
Other:
- moved on the sheet: R13, R14, R16, R17, R18, R19, R21, R22, R23, R24, R25
