File: HatBoard/hat_board.kicad_sch (KiCad schematic)
At the start: 0 parts

Commit message: new everything should be here
Parts:
- added C16, C17: 1uF, Capacitor_SMD:C_0805_2012Metric, symbol Device:C
- added C18: 100nF, Capacitor_SMD:C_0402_1005Metric, symbol Device:C
- added C39: 10nF, Capacitor_SMD:C_0402_1005Metric, symbol Device:C
- added D1, D2, D3, D4: D_Schottky, easyeda2kicad:POWERDI-123_L2.8-W1.8-LS3.7-RD, symbol Device:D_Schottky
- added J2: Conn_01x04, Connector_PinHeader_2.00mm:PinHeader_1x04_P2.00mm_Vertical, symbol Connector_Generic:Conn_01x04
- added J3: DF11 FC Connection, easyeda2kicad:CONN-TH_DF11-12DS-2DSA-05, symbol Connector_Generic:Conn_02x03_Odd_Even
- added J4, J5, J6: DF11 FC Connection, easyeda2kicad:CONN-TH_DF11-12DS-2DSA-05, symbol Connector_Generic:Conn_02x06_Odd_Even
- added R1, R2: 10K, Resistor_SMD:R_0603_1608Metric, symbol Device:R_US
- added R15: 57.2, Resistor_SMD:R_0603_1608Metric, symbol Device:R_US
- added U10: VEML7700, easyeda2kicad:SENSOR-SMD_EML7700-TT, symbol Adafruit VEML7700-eagle-import:VEML7700
- added U12: DRV2605LDGS, Package_SO:VSSOP-10_3x3mm_P0.5mm, symbol Driver_Haptic:DRV2605LDGS
- added U27: TMP112AIDRLR, easyeda2kicad:SOT-563_L1.6-W1.2-P0.50-LS1.6-BR, symbol easyeda2kicad:TMP112AIDRLR
Connections:
- new net: D2.1 (K), J4.6 (Pin_6)
- new net: C17.1, U12.1 (REG)
- new net: R15.1, U12.7 (OUT+)
- new net: R15.2, U12.9 (OUT-)
- new net: D4.1 (K), J6.10 (Pin_10), J6.4 (Pin_4)
- new net: D1.1 (K), J3.4 (Pin_4)
- new net: D3.1 (K), J5.10 (Pin_10), J5.4 (Pin_4)
- new net +3V3: C16.1, C18.1, C39.1, D1.2 (A), D2.2 (A), D3.2 (A), D4.2 (A), R1.2, R2.2, U10.2 (VDD), U12.10 (VDD), U12.5 (EN), U27.5 (V+)
- new net GND: C16.2, C17.2, C18.2, C39.2, J2.1 (Pin_1), J2.4 (Pin_4), J3.5 (Pin_5), J4.11 (Pin_11), J4.12 (Pin_12), J5.11 (Pin_11), J5.5 (Pin_5), J6.11 (Pin_11), J6.5 (Pin_5), U10.3 (GND), U12.4 (IN/TRIG), U12.8 (GND), U27.2 (GND), U27.4 (ADD0)
- new net SCDAIN_F4: J5.12 (Pin_12)
- new net SCL: J2.2 (Pin_2), R2.1, U10.1 (SCL), U12.2 (SCL), U27.1 (SCL)
- new net SCLINZ: J3.6 (Pin_6)
- new net SCLIN_ANT: J4.7 (Pin_7)
- new net SCLIN_F1: J6.6 (Pin_6)
- new net SCLIN_F2: J6.8 (Pin_8)
- new net SCLIN_F3: J5.6 (Pin_6)
- new net SCLIN_F4: J5.8 (Pin_8)
- new net SDA: J2.3 (Pin_3), R1.1, U10.4 (SDA), U12.3 (SDA), U27.6 (SDA)
- new net SDAINZ: J3.2 (Pin_2)
- new net SDAIN_ANT: J4.5 (Pin_5)
- new net SDAIN_F1: J6.2 (Pin_2)
- new net SDAIN_F2: J6.12 (Pin_12)
- new net SDAIN_F3: J5.2 (Pin_2)
- no-connect marks 0 -> 19
Other:
- sheet Face Board4 renamed Z-Board
- sheet Face Board5 renamed Antenna Board
- sheet Antenna Board ports: added SCLIN, SDAIN; removed none
- sheet Face Board ports: added SCLIN, SDAIN; removed none
- sheet Face Board1 ports: added SCLIN, SDAIN; removed none
- sheet Face Board2 ports: added SCLIN, SDAIN; removed none
- sheet Face Board3 ports: added SCLIN, SDAIN; removed none
- sheet Z-Board ports: added SCLIN, SDAIN; removed none
- note added: "Bus Pullup resistors"
- note added: "Haptic Motor Driver"
- note added: "Light Sensor"
- note added: "Temperature Sensor"
